File: LCD_Adapter/LCD_Adapter/LCD_Adapter.kicad_pcb (KiCad board)
At the start: 4 copper layers, 47 x 75 mm, 42 parts, among them J1 Conn_01x10, J2 FH12-30S-0.5SH_55_, J3 Conn_01x22, J4 1-1734248-5, J5 FH12-30S-0.5SH_55_, U1 TLV75801PDBV, U2 TLV75801PDBV, U3 TPS61042DRBR

Commit message: PCB_UPDATE
Parts:
- removed J3: Conn_01x22, lib:FC-10A20P11H20
- added C10: 100nF, Capacitor_SMD:C_0402_1005Metric, F.Cu at (109.7, 72.4)
- added C11: 100nF, Capacitor_SMD:C_0402_1005Metric, F.Cu at (114.8, 73.8)
- added C12: 100nF, Capacitor_SMD:C_0402_1005Metric, F.Cu at (114.8, 76.2)
- added C9: 100nF, Capacitor_SMD:C_0402_1005Metric, F.Cu at (109.8, 74.7)
- added J6: 2-1734248-0, lib:2-1734248-0, F.Cu at (101.2, 78.0)
- added R10: 10k, Resistor_SMD:R_0603_1608Metric, F.Cu at (121.0, 47.0)
- added R11: 10k, Resistor_SMD:R_0603_1608Metric, F.Cu at (108.6, 54.5)
- added R6: 10k, Resistor_SMD:R_0603_1608Metric, F.Cu at (121.0, 55.6)
- added R7: 10k, Resistor_SMD:R_0603_1608Metric, F.Cu at (121.0, 57.1)
- added R8: 10k, Resistor_SMD:R_0603_1608Metric, F.Cu at (121.0, 54.1)
- added R9: 10k, Resistor_SMD:R_0603_1608Metric, F.Cu at (121.0, 48.6)
- moved J2 5.21 mm to (127.5, 65.2)
- moved TP4 3.93 mm to (108.2, 66.0)
- moved TP3 3.19 mm to (108.2, 64.0)
- moved TP2 1.86 mm to (108.2, 68.0)
- moved R3 0.05 mm to (108.6, 56.0)
Connections:
- J2 pad 1:  LED_A -> LCM_ID
- J2 pad 10: /STM2LCD/D0_P -> GND
- J2 pad 11: /STM2LCD/D0_N -> /STM2LCD/D2_N
- J2 pad 12: GND -> /STM2LCD/D2_P
- J2 pad 13: /STM2LCD/D1_P -> GND
- J2 pad 14: /STM2LCD/D1_N -> /STM2LCD/CLK_N
- J2 pad 15: GND -> /STM2LCD/CLK_P
- J2 pad 16: /STM2LCD/CLK_P -> GND
- J2 pad 17: /STM2LCD/CLK_N -> /STM2LCD/D1_N
- J2 pad 18: GND -> /STM2LCD/D1_P
- J2 pad 19: /STM2LCD/D2_P -> GND
- J2 pad 2:  LED_K -> +2V8
- J2 pad 20: /STM2LCD/D2_N -> /STM2LCD/D0_N
- J2 pad 21: GND -> /STM2LCD/D0_P
- J2 pad 22: /STM2LCD/D3_P -> GND
- J2 pad 23: /STM2LCD/D3_N -> PWM
- J2 pad 24: GND -> TE
- J2 pad 25: TP_INT -> RESET
- J2 pad 26: TP_SDA -> +1V8
- J2 pad 27: TP_SCL -> +2V8
- J2 pad 28: TP_RES ->  LED_K
- J2 pad 29: +2V8 ->  LED_K
- J2 pad 3:  LED_K -> TP_RES
- J2 pad 30: LCM_ID ->  LED_A
- J2 pad 4: +2V8 -> TP_SCL
- J2 pad 5: +1V8 -> TP_SDA
- J2 pad 6: RESET -> TP_INT
- J2 pad 7: TE -> GND
- J2 pad 8: PWM -> /STM2LCD/D3_N
- J2 pad 9: GND -> /STM2LCD/D3_P
- J5 pad 1:  LED_A -> LCM_ID
- J5 pad 10: /RPI2LCD/RPI_D0_P -> GND
- J5 pad 11: /RPI2LCD/RPI_D0_N -> /RPI2LCD/RPI_D2_N
- J5 pad 12: GND -> /RPI2LCD/RPI_D2_P
- J5 pad 13: /RPI2LCD/RPI_D1_P -> GND
- J5 pad 14: /RPI2LCD/RPI_D1_N -> /RPI2LCD/RPI_CLK_N
- J5 pad 15: GND -> /RPI2LCD/RPI_CLK_P
- J5 pad 16: /RPI2LCD/RPI_CLK_P -> GND
- J5 pad 17: /RPI2LCD/RPI_CLK_N -> /RPI2LCD/RPI_D1_N
- J5 pad 18: GND -> /RPI2LCD/RPI_D1_P
- J5 pad 19: /RPI2LCD/RPI_D2_P -> GND
- J5 pad 2:  LED_K -> +2V8
- J5 pad 20: /RPI2LCD/RPI_D2_N -> /RPI2LCD/RPI_D0_N
- J5 pad 21: GND -> /RPI2LCD/RPI_D0_P
- J5 pad 22: /RPI2LCD/RPI_D3_P -> GND
- J5 pad 23: /RPI2LCD/RPI_D3_N -> PWM
- J5 pad 24: GND -> TE
- J5 pad 25: TP_INT -> RESET
- J5 pad 26: RPI_TP_SDA -> +1V8
- J5 pad 27: RPI_TP_SCL -> +2V8
- J5 pad 28: TP_RES ->  LED_K
- J5 pad 29: +2V8 ->  LED_K
- J5 pad 3:  LED_K -> TP_RES
- J5 pad 30: LCM_ID ->  LED_A
- J5 pad 4: +2V8 -> RPI_TP_SCL
- J5 pad 5: +1V8 -> RPI_TP_SDA
- J5 pad 6: RESET -> TP_INT
- J5 pad 7: TE -> GND
- J5 pad 8: PWM -> /RPI2LCD/RPI_D3_N
- J5 pad 9: GND -> /RPI2LCD/RPI_D3_P
Routing:
- net TE: track 65.5 -> 32.0 mm, vias 3 -> 4
- net /STM2LCD/CLK_N: track 53.5 -> 32.5 mm, vias 0 -> 2
- net /STM2LCD/CLK_P: track 53.1 -> 32.4 mm, vias 0 -> 2
- net /STM2LCD/D0_N: track 52.9 -> 34.4 mm
- net /STM2LCD/D0_P: track 53.2 -> 35.0 mm
- net /STM2LCD/D1_N: track 53.0 -> 35.2 mm
- net /STM2LCD/D1_P: track 53.1 -> 35.9 mm
- net +1V8: track 74.7 -> 89.0 mm, vias 7 -> 9
- net TP_RES: track 55.6 -> 69.9 mm, vias 4 -> 2
- net LCM_ID: track 75.0 -> 86.8 mm
- net PWM: track 60.8 -> 49.8 mm, vias 4 -> 3
- net TP_SDA: track 26.9 -> 34.7 mm
- net GND: track 85.9 -> 79.8 mm, vias 100 -> 90
- net TP_INT: track 74.4 -> 68.5 mm, vias 4 -> 3
- net Net-(J6-Pad20): track 4.85 -> 9.09 mm
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