File: LCD_Adapter/LCD_Adapter/RPI2LCD.kicad_sch (KiCad schematic)
At the start: 5 parts, among them J4 1-1734248-5, J5 FH12-30S-0.5SH_55_

Commit message: PCB_UPDATE
Parts:
- added C10, C11, C12, C9: 100nF, Capacitor_SMD:C_0402_1005Metric, symbol Device:C
Connections:
- net  LED_A: now also J5.30; no longer J5.1
- net  LED_K: now also J5.28, J5.29; no longer J5.2, J5.3
- net +1V8: now also J5.26; no longer J5.5
- net +2V8: now also J5.2, J5.27; no longer J5.29, J5.4
- net +3V3: now also C10.1, C11.1, C12.1, C9.1
- net GND: now also J5.10, J5.13, J5.16, J5.19, J5.22, J5.7, C10.2, C11.2, C12.2, C9.2; no longer J5.12, J5.15, J5.18, J5.21, J5.24, J5.9
- net LCM_ID: now also J5.1; no longer J5.30
- net PWM: now also J5.23; no longer J5.8
- net RESET: now also J5.25; no longer J5.6
- net RPI_CLK_N: now also J5.14; no longer J5.17
- net RPI_CLK_P: now also J5.15; no longer J5.16
- net RPI_D0_N: now also J5.20; no longer J5.11
- net RPI_D0_P: now also J5.21; no longer J5.10
- net RPI_D1_N: now also J5.17; no longer J5.14
- net RPI_D1_P: now also J5.18; no longer J5.13
- net RPI_D2_N: now also J5.11; no longer J5.20
- net RPI_D2_P: now also J5.12; no longer J5.19
- net RPI_D3_N: now also J5.8; no longer J5.23
- net RPI_D3_P: now also J5.9; no longer J5.22
- net RPI_TP_SCL: now also J5.4; no longer J5.27
- net RPI_TP_SDA: now also J5.5; no longer J5.26
- net TE: now also J5.24; no longer J5.7
- net TP_INT: now also J5.6; no longer J5.25
- net TP_RES: now also J5.3; no longer J5.28
Other:
- moved on the sheet: J5
