File: LCD_Adapter/LCD_Adapter/STM2LCD.kicad_sch (KiCad schematic)
At the start: 11 parts, among them J1 Conn_01x10, J2 FH12-30S-0.5SH_55_, J3 Conn_01x22

Commit message: PCB_UPDATE
Parts:
- removed J3: Conn_01x22, lib:FC-10A20P11H20, symbol Connector_Generic:Conn_01x22
- added J6: 2-1734248-0, CONN_2-1734248-0_TYCO, symbol 2-1734248-0:2-1734248-0
- added R10, R11, R6, R7, R8, R9: 10k, Resistor_SMD:R_0603_1608Metric, symbol Device:R
- R2, R3, R4, R5: now not fitted
Connections:
- net  LED_A: now also J2.30; no longer J2.1
- net  LED_K: now also J2.28, J2.29; no longer J2.2, J2.3
- net +1V8: now also J2.26, R8.2, R9.2; no longer J2.5
- net +2V8: now also J2.2, J2.27, R10.2, R6.2; no longer J2.29, J2.4
- net +3V3: now also J6.14, J6.15, J6.34, J6.35
- net CLK_N: now also J2.14, J6.25, J6.5; no longer J2.17
- net CLK_P: now also J2.15, J6.26, J6.6; no longer J2.16
- net D0_N: now also J2.20, J6.28, J6.8; no longer J2.11
- net D0_P: now also J2.21, J6.29, J6.9; no longer J2.10
- net D1_N: now also J2.17, J6.2, J6.22; no longer J2.14
- net D1_P: now also J2.18, J6.23, J6.3; no longer J2.13
- net D2_N: now also J2.11; no longer J2.20
- net D2_P: now also J2.12; no longer J2.19
- net D3_N: now also J2.8; no longer J2.23
- net D3_P: now also J2.9; no longer J2.22
- net GND: now also J2.10, J2.13, J2.16, J2.19, J2.22, J2.7, J6.1, J6.10, J6.13, J6.16, J6.21, J6.24, J6.27, J6.30, J6.33, J6.36, J6.4, J6.7, R11.1, R7.1; no longer J2.12, J2.15, J2.18, J2.21, J2.24, J2.9
- net LCM_ID: now also J2.1; no longer J2.30
- net PWM: now also J2.23; no longer J2.8
- net RESET: now also J2.25, R10.1, R11.2, R9.1; no longer J2.6
- net TE: now also J2.24; no longer J2.7
- net TP_INT: now also J2.6; no longer J2.25
- net TP_RES: now also J2.3, R6.1, R7.2, R8.1; no longer J2.28
- net TP_SCL: now also J2.4, J6.11, J6.31; no longer J2.27
- net TP_SDA: now also J2.5, J6.12, J6.32; no longer J2.26
- net at R1.1: now also J6.19, J6.39
- net at R5.1: now also J6.17, J6.37
- net at R4.1: now also J6.18, J6.38
- net at R2.1, R3.1: now also J6.20, J6.40
Other:
- moved on the sheet: J2
