File: PCB/MPU_MOD.kicad_pcb (KiCad board)
At the start: 8 copper layers, 43.5 x 70 mm, 305 parts, among them J1 SJ-43504-SMT-TR, J2 2-1734248-0, J3 USB4510-03-1-A_REVA, J501 MEM2090-00-145-00-A_REVA, J701 FTSH-107-01-L-DV-K-A, J901 73412-0110, U1 IS21ES08GA-JQLI-TR, U201 STC3115IQT, U203 STPMIC1APQR, U3 BQ24298RTWR, U301 STM32MP157FABx, U401 MT41K256M16TW-107_P, U502 HSP051-4M10, U503 HSP051-4M10, U701 HSP051-4M10, U702 HSP051-4M10, U801 FUSB302BMPX, U802 HSP051-4M10, U901 LBEE5PK2AE-771, Y601 NX2012SA-32.768K, Y701 ECS-2520MVQ-240

Commit message: PCB_UPDATE
Parts:
- moved C429 12.2 mm to (98.9, 63.2), turned to 180 degrees
- moved C403 3.06 mm to (99.6, 60.2)
- moved R403 1.69 mm to (103.6, 72.0), turned to 45 degrees
- moved C427 0.66 mm to (107.8, 72.7), turned to -45 degrees
- moved R404 0.57 mm to (100.5, 73.4), turned to 0 degrees
Routing:
- net /DDR/DDR_DQ14: track 39.2 -> 20.7 mm
- net /DDR/DDR_RESETN: track 0.00 -> 13.3 mm, vias 0 -> 1
- net GND: track 67.2 -> 77.6 mm, vias 89 -> 96
- net /DDR/DDR_A12: track 25.3 -> 33.5 mm
- net /DDR/DDR_A1: track 23.6 -> 30.4 mm
- net /DDR/DDR_A10: track 23.3 -> 29.8 mm
- net /DDR/DDR_BA2: track 30.2 -> 24.0 mm
- net VDD_DDR: track 16.1 -> 21.4 mm, vias 14 -> 19
- net /DDR/DDR_A14: track 23.2 -> 28.2 mm
- net /DDR/DDR_A0: track 29.1 -> 24.2 mm
- net /DDR/DDR_CSN: track 27.6 -> 32.4 mm
- net /DDR/DDR_A11: track 27.6 -> 32.1 mm
- net /DDR/DDR_ODT: track 25.7 -> 30.0 mm
- net Net-(U401-ZQ): track 0.00 -> 4.03 mm
- net /DDR/DDR_A2: track 27.3 -> 23.6 mm
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
Commit message: PCB_UPDATE
Parts:
- moved C427 2.80 mm to (110.6, 73.2)
- moved R419 2.49 mm to (97.3, 63.1)
- moved C422 1.83 mm to (108.8, 62.3)
- moved R415 1.50 mm to (99.3, 63.1)
- moved R421 1.50 mm to (104.0, 63.1)
- moved C409 1.50 mm to (99.0, 61.0)
- moved C410 1.50 mm to (100.9, 61.0)
- moved C411 1.50 mm to (102.9, 61.0)
- moved C413 1.50 mm to (106.8, 61.1)
- moved C414 1.50 mm to (104.9, 61.1)
- moved R406 1.50 mm to (103.1, 63.1)
- moved R408 1.50 mm to (101.2, 63.1)
- moved R409 1.50 mm to (102.1, 63.1)
- moved R411 1.50 mm to (100.2, 63.1)
- moved R423 1.50 mm to (105.0, 63.1)
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Routing:
- net VDD_DDR: track 21.4 -> 33.5 mm, vias 19 -> 25
- net GND: track 77.6 -> 88.9 mm, vias 96 -> 102
- net /DDR/DDR_BA2: track 24.0 -> 30.1 mm
- net /DDR/DDR_A0: track 24.2 -> 29.3 mm
- net /DDR/DDR_BA0: track 23.9 -> 28.1 mm
- net /DDR/DDR_A2: track 23.6 -> 27.3 mm
- net /DDR/DDR_A9: track 25.2 -> 28.4 mm
- net /DDR/DDR_A3: track 23.3 -> 26.4 mm
- net /DDR/DDR_CLK_P: track 23.8 -> 26.5 mm
- net /DDR/DDR_CSN: track 32.4 -> 29.7 mm
- net /DDR/DDR_A5: track 25.4 -> 27.8 mm
- net /DDR/DDR_ODT: track 30.0 -> 28.1 mm
- net /DDR/DDR_CLK_N: track 23.9 -> 25.7 mm
- net /DDR/DDR_CKE: track 19.8 -> 21.0 mm
- net VREF_DDR: track 6.21 -> 7.25 mm
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
Commit message: added step file
Parts:
- moved S602 40.8 mm to (110.5, 36.3), turned to 90 degrees
- moved J501 1.32 mm to (112.0, 48.7)
