File: PCB/MPU_MOD.kicad_pcb (KiCad board)
At the start: 6 copper layers, 43.5 x 95 mm, 277 parts, among them J1 MEM2090-00-145-00-A_REVA, J2 FTSH-107-01-L-DV-K-A, J4 Conn_02x15_Odd_Even, J5 SFV30R-4STBE1HLF, J6 USB4510-03-1-A_REVA, Q1 CSD23381F4, U11 SIS903DN-T1-GE3, U12 STUSB1600AQTR, U13 HSP051-4M10, U14 SIS903DN-T1-GE3, U15 BQ25887RGER, U16 TPS563252DRLR, U3 STPMIC1APQR, U4 STM32MP157FABx, U5 MT41K256M16TW-107_P, U6 HSP051-4M10, U7 HSP051-4M10, U8 HSP051-4M10, U9 HSP051-4M10, Y1 NX2012SA-32.768K, Y2 ECS-2520MVQ-240

Commit message: Update MPU_MOD.kicad_pcb
Parts:
- moved L7 19.4 mm to (23.6, 69.5), turned to 180 degrees
- moved C132 13.6 mm to (27.6, 73.5), turned to -90 degrees
- moved C127 11.2 mm to (20.9, 72.0)
- moved C128 10.8 mm to (23.2, 71.7), turned to 180 degrees
- moved U15 9.08 mm to (22.4, 75.0)
- moved C135 0.43 mm to (1.80, 90.9)
- moved R85 0.43 mm to (1.80, 89.2)
- moved L8 0.43 mm to (1.35, 93.5)
- moved C133 0.43 mm to (4.40, 88.3)
- moved C136 0.43 mm to (4.65, 95.4)
- moved C137 0.43 mm to (3.95, 94.2)
- moved R86 0.43 mm to (7.70, 92.2)
- moved U16 0.43 mm to (4.65, 92.5)
- moved R84 0.43 mm to (1.80, 90.1)
- moved C134 0.43 mm to (4.40, 90.3)
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
Commit message: pcb update
Parts:
- removed BT2, BT3: Battery_Cell, Connector_PinHeader_1.00mm:PinHeader_1x02_P1.00mm_Vertical
- removed C123, C124, C125, C126, C127: 1uF, lib:C_0402_small
- removed C128, C131: 10uF, Capacitor_SMD:C_0603_1608Metric
- removed C129: 4.7nF, lib:C_0402_small
- removed C130: 4.7uF, lib:C_0402_small
- removed C132: 47uF, Capacitor_SMD:C_1206_3216Metric
- removed C133, C134: 10uF, Capacitor_SMD:C_0805_2012Metric
- removed C135, C137: 100nF, lib:C_0402_small
- removed C136: 22uF, Capacitor_SMD:C_0603_1608Metric
- removed D10: LED, LED_SMD:LED_0402_1005Metric
- removed H1, H2, H3, H4: MountingHole_Pad, MountingHole:MountingHole_2.7mm_M2.5_Pad_Via
- removed J4: Conn_02x15_Odd_Even, Connector_PinHeader_2.54mm:PinHeader_2x15_P2.54mm_Horizontal
- removed L7: 1uH, Inductor_SMD:L_1008_2520Metric
- removed L8: IHLP1210BZEZ3R3M5A, lib:IHLP1210BZEZ_VIS
- removed R13: 0, Resistor_SMD:R_0805_2012Metric
- removed R71, R73: 1k, lib:R_0402_small
- removed R72, R74, R75, R76, R82: 10k, lib:R_0402_small
- removed R77: 330, lib:R_0402_small
- removed R78: 9.5, lib:R_0402_small
- removed R79: 5.23k, lib:R_0402_small
- removed R80: 30.1k, lib:R_0402_small
- removed R81: 1k, Resistor_SMD:R_0402_1005Metric
- removed R83: 383, lib:R_0402_small
- removed R84: 100k, lib:R_0402_small
- removed R85: 25.5k, lib:R_0402_small_RES
- removed R86: 220k, lib:R_0402_small
- removed R87: 30k, lib:R_0402_small
- removed S2, S3, S4: EVQ-9P701P, lib:SW_EVQ-9P701P
- removed TH2: Thermistor, Connector_PinHeader_1.00mm:PinHeader_1x02_P1.00mm_Vertical
- removed TP10, TP11, TP12, TP13, TP14, TP15, TP16, TP17, TP18, TP19, TP20, TP28, TP29, TP30, TP31, TP32, TP33, TP34, TP35, TP36, TP37, TP4, TP5, TP6, TP7, TP8, TP9: TestPoint, lib:TP_0.5
- removed U11, U14: SIS903DN-T1-GE3, lib:SIS309
- removed U12: STUSB1600AQTR, lib:QFN50P400X400X100-25N
- removed U15: BQ25887RGER, lib:IC_BQ25887RGER
- removed U16: TPS563252DRLR, lib:TPS563252DRLR
- moved R56 58.9 mm to (23.6, 127.4)
- moved R57 58.9 mm to (22.6, 127.4)
- moved C122 39.1 mm to (84.7, 116.5)
- moved C120 35.6 mm to (85.0, 117.8), turned to 180 degrees
- moved C121 35.6 mm to (85.0, 118.6)
- moved D9 35.2 mm to (85.0, 119.9), turned to 180 degrees
- moved L5 13.1 mm to (73.8, 101.4)
- moved C16 13.1 mm to (77.8, 103.0)
- moved C18 13.1 mm to (67.8, 105.5)
- moved C19 13.1 mm to (77.8, 107.5)
- moved C23 13.1 mm to (67.8, 106.5)
- moved C24 13.1 mm to (77.8, 104.8)
- moved L2 13.1 mm to (70.2, 112.0)
- moved L3 13.1 mm to (74.9, 112.7)
- moved L4 13.1 mm to (69.7, 101.4)
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Connections:
- C120 pad 1: VIN_USB -> VIN
- C121 pad 2: VIN_USB -> VIN
- C122 pad 2: VIN_USB -> VIN
- D9 pad 1: VIN_USB -> VIN
- J6 pad A4_B9: VIN_USB -> VIN
- J6 pad B4_A9: VIN_USB -> VIN
- U4 pad B5: uSD_DETECT -> I2C1_SDA
- U4 pad W6: unconnected-(U4C-PB8-PadW6) -> I2C1_SCL
Routing:
- net USB_M_D+: track 31.5 -> 0.00 mm
- net USB_M_D-: track 30.0 -> 0.00 mm
- net USB_D-: track 31.8 -> 50.2 mm, vias 0 -> 3
- net USB_D+: track 31.4 -> 49.7 mm, vias 0 -> 3
- net FDCAN2_RX: track 16.9 -> 0.57 mm, vias 2 -> 1
- net I2S3_WS: track 13.5 -> 0.05 mm
- net ETH1_TX_EN: track 13.4 -> 0.04 mm, vias 2 -> 0
- net FDCAN2_TX: track 13.4 -> 1.10 mm, vias 2 -> 1
- net I2S2_WS: track 12.9 -> 0.56 mm
- net UART7_RX_STM: track 12.5 -> 1.09 mm, vias 2 -> 1
- net UART7_TX_STM: track 12.1 -> 1.13 mm, vias 2 -> 1
- net I2S2_CK: track 11.4 -> 0.62 mm
- net I2S3_SDO: track 10.7 -> 0.03 mm
- net I2S2_SDI: track 11.3 -> 0.66 mm
- net I2S3_CK: track 10.6 -> 0.00 mm
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- added copper zone on In1.Cu, net GND
Other:
- board size 43.5 x 95 mm -> 50 x 70 mm
