File: PCB/MPU_PWR.kicad_sch (KiCad schematic)
At the start: 41 parts, among them U301 STM32MP157FABx

Commit message: PCB_UPDATE
Parts:
- added C1, C2, C3, C4, C5, C6, C7: 1uF, lib:C_0402_small, symbol Device:C
- added C8, C9: 1nF, lib:C_0402_small, symbol Device:C
Connections:
- net GND: now also C1.1, C2.1, C3.1, C4.1, C5.1, C6.1, C7.1, C8.1, C9.1
- net VDD: now also C1.2, C2.2, C3.2, C4.2, C5.2
- net VDD_CORE: now also C6.2, C7.2
- net VDD_DDR: now also C8.2, C9.2
Other:
- moved on the sheet: C320, C321, C322, C323, C324, C325
