File: PCB/MPU_PWR.kicad_sch (KiCad schematic)
At the start: 47 parts, among them U4 STM32MP157FABx

Commit message: PCB_UPDATE
Parts:
- C31, C32, C33, C34, C38, C39, C40, C41, C42, C43, C44, C45, C46, C47, C48, C49, C50, C51, C52, C53, C54, C55, C56, C57, C58, C59, C60, C65, C67, C68, C69, C70, C72, C74, C76: LCSC Part # (none) -> C52923; P/N GRM155R61E105KA12D -> (none); REC P/N (none) -> GRM155R61E105KA12D
- C61, C62, C63, C64: LCSC Part # (none) -> C1523; P/N GRM155R70J102KA01D -> (none); REC P/N (none) -> GRM155R70J102KA01D
- C66, C78: LCSC Part # (none) -> C307331; P/N GRM155R61E104KA87J -> (none); REC P/N (none) -> GRM155R61E104KA87J
- C73, C75, C77: LCSC Part # (none) -> C12530; P/N GRT153R60J225ME13D -> (none); REC P/N (none) -> GRT153R60J225ME13D
- L6: LCSC Part # (none) -> C76799; P/N MLZ1608M4R7WT000 -> (none); REC P/N (none) -> MLZ1608M4R7WT000
- U4: LCSC Part # (none) -> C1236734

Commit message: UPDATE
Parts:
- renumbered C31 to C301, C32 to C302, C33 to C303, C34 to C304, C38 to C305, C39 to C306, C40 to C307, C41 to C308, C42 to C309, C43 to C310, C44 to C311, C45 to C312, C46 to C313, C47 to C314, C48 to C315, C49 to C316, C50 to C317, C51 to C318, C52 to C319, C53 to C320, C54 to C321, C55 to C322, C56 to C323, C57 to C324, C58 to C325, C59 to C326, C60 to C327, C61 to C328, C62 to C329, C63 to C330, C64 to C331, C65 to C332, C66 to C333, C67 to C334, C68 to C335, C69 to C336, C70 to C337, C71 to C338, C72 to C339, C73 to C340, C74 to C341, C75 to C342, C76 to C343, C77 to C344, C78 to C345, L6 to L301
