File: PCB/PWR.kicad_sch (KiCad schematic)
At the start: 68 parts, among them U201 STC3115IQT, U203 STPMIC1APQR, U3 BQ24298RTWR

Commit message: PCB_UPDATE
Parts:
- D203: value PTVS3V3S1UR -> MSP3V3-M3/89A; footprint lib:TVS_PTVS3V3S1UR -> Diode_SMD:D_MicroSMP_KA; MAXIMUM_PACKAGE_HEIGHT 1.1 mm -> (none); MP PTVS3V3S1UR -> (none)
- TP201, TP202, TP203, TP204, TP205, TP206, TP207, TP208, TP209, TP210, TP211, TP212: footprint Library:TP_0.5mm -> lib:TP_0.5
Connections:
- net GND: now also D203.2; no longer D203.A
- net PWR_SW_WAKE_UP: now also D203.1; no longer D203.C
Changed lines of the file:
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@@
 			)
 		)
-		(property "Footprint" "Library:TP_0.5mm"
+		(property "Footprint" "lib:TP_0.5"
 			(at 382.27 191.77 0)
 			(effects
@@
 			)
 		)
-		(property "Value" "PTVS3V3S1UR"
+		(property "Value" "MSP3V3-M3/89A"
 			(at 254 255.2699 90)
 			(effects
@@
 			)
 		)
-		(property "Footprint" "lib:TVS_PTVS3V3S1UR"
+		(property "Footprint" "Diode_SMD:D_MicroSMP_KA"
 			(at 256.54 254 0)
 			(effects
@@
 			)
 		)
-		(property "MAXIMUM_PACKAGE_HEIGHT" "1.1 mm"
+		(property "MAXIMUM_PACKAGE_HEIGHT" ""
 			(at 256.54 254 0)
 			(effects
@@
 			)
 		)
-		(property "MP" "PTVS3V3S1UR"
+		(property "MP" ""
 			(at 256.54 254 0)
 			(effects
@@
 			)
 		)
-		(pin "C"
+		(pin "2"
 		)
-		(pin "A"
+		(pin "1"
 		)
 		(instances
@@
 			)
 		)
-		(property "Footprint" "Library:TP_0.5mm"
+		(property "Footprint" "lib:TP_0.5"
 			(at 170.18 229.87 0)
 			(effects
@@
 			)
 		)
-		(property "Footprint" "Library:TP_0.5mm"
+		(property "Footprint" "lib:TP_0.5"
 			(at 382.27 205.74 0)
 			(effects
@@
 			)
 		)
-		(property "Footprint" "Library:TP_0.5mm"
+		(property "Footprint" "lib:TP_0.5"
 			(at 34.29 128.27 0)
 			(effects
@@
 			)
 		)
-		(property "Footprint" "Library:TP_0.5mm"
+		(property "Footprint" "lib:TP_0.5"
 			(at 382.27 219.71 0)
 			(effects
@@
 			)
 		)
-		(property "Footprint" "Library:TP_0.5mm"
+		(property "Footprint" "lib:TP_0.5"
 			(at 303.53 35.56 0)
 			(effects
@@
 			)
 		)
-		(property "Footprint" "Library:TP_0.5mm"
+		(property "Footprint" "lib:TP_0.5"
 			(at 391.16 77.47 0)
 			(effects
@@
 			)
 		)
-		(property "Footprint" "Library:TP_0.5mm"
+		(property "Footprint" "lib:TP_0.5"
 			(at 381 149.86 0)
 			(effects
@@
 			)
 		)
-		(property "Footprint" "Library:TP_0.5mm"
+		(property "Footprint" "lib:TP_0.5"
 			(at 391.16 35.56 0)
 			(effects
@@
 			)
 		)
-		(property "Footprint" "Library:TP_0.5mm"
+		(property "Footprint" "lib:TP_0.5"
 			(at 391.16 63.5 0)
 			(effects
@@
 			)
 		)
-		(property "Footprint" "Library:TP_0.5mm"
+		(property "Footprint" "lib:TP_0.5"
 			(at 391.16 49.53 0)
 			(effects
@@
 			)
 		)
-		(property "Footprint" "Library:TP_0.5mm"
+		(property "Footprint" "lib:TP_0.5"
 			(at 34.29 130.81 0)
 			(effects
