File: PCB/PWR.kicad_sch (KiCad schematic)
At the start: 47 parts, among them Q1 CSD23381F4, U10 TPS62840DLCR, U3 STPMIC1APQR

Commit message: UPDATE
Parts:
- renumbered C118 to C201, C117 to C202, C10 to C203, C11 to C204, C12 to C205, C13 to C206, C14 to C207, C15 to C208, C16 to C209, C17 to C210, C18 to C211, C19 to C212, C20 to C213, C21 to C214, C22 to C215, C23 to C216, C24 to C217, C25 to C218, C26 to C219, C27 to C220, C28 to C221, C29 to C222, C30 to C223, D3 to D201, L7 to L201, L2 to L202, L3 to L203, L4 to L204, L5 to L205, Q1 to Q201, R47 to R201, R15 to R202, R16 to R203, S1 to S201, TP4 to TP201, TP5 to TP202, TP1 to TP203, TP6 to TP204, TP7 to TP205, TP8 to TP206, TP2 to TP207, TP9 to TP208, TP10 to TP209, TP11 to TP210, TP12 to TP211, U10 to U201, U3 to U202

Commit message: UPDATE
Parts:
- Q201: value CSD23381F4 -> DMG1013T-7; footprint lib:CSD23381F4 -> Package_TO_SOT_SMD:SOT-523; LCSC Part # C129355 -> (none)
Other:
- note added: "ENABLE later than 1.15 ms after 3.3V"
Changed lines of the file:
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@@
 		)
 	)
+	(text "ENABLE later than  1.15 ms after 3.3V"
+		(exclude_from_sim no)
+		(at 70.104 55.88 0)
+		(effects
+			(font
+				(size 1.27 1.27)
+			)
+		)
+	)
 	(text "120mA LDO max\n"
 		(exclude_from_sim no)
@@
 			)
 		)
-		(property "Value" "CSD23381F4"
+		(property "Value" "DMG1013T-7"
 			(at 261.62 207.0101 0)
 			(effects
@@
 			)
 		)
-		(property "Footprint" "lib:CSD23381F4"
+		(property "Footprint" "Package_TO_SOT_SMD:SOT-523"
 			(at 260.35 210.82 0)
 			(effects
@@
 			)
 		)
-		(property "LCSC Part #" "C129355"
+		(property "LCSC Part #" ""
 			(at 255.27 208.28 0)
 			(effects

Commit message: UPDATE
Parts:
- removed S201: EVQ-9P701P, lib:SW_EVQ-9P701P, symbol EVQ-9P701P:EVQ-9P701P
- added S2: B3U-3000P, lib:SW_B3U-3000P, symbol B3U-3000P:B3U-3000P
Connections:
- net GND: now also S2.2
- net at C203.2, D201.1, U202.17 (~{PONKEY}): now also S2.1
