File: PCB/RCC_BOOT_RST_DEBUG.kicad_sch (KiCad schematic)
At the start: 36 parts, among them J701 FTSH-107-01-L-DV-K-A, U301 STM32MP157FABx, U701 HSP051-4M10, U702 HSP051-4M10, Y701 ECS-2520MVQ-240

Commit message: PCB_UPDATE
Parts:
- removed D701: PTVS3V3S1UR, lib:TVS_PTVS3V3S1UR, symbol PTVS3V3S1UR:PTVS3V3S1UR
- added D3: MSP3V3-M3/89A, Diode_SMD:D_MicroSMP_KA, symbol PTVS3V3S1UR:PTVS3V3S1UR
- TP701, TP702, TP703, TP704, TP705, TP706, TP707, TP708, TP709, TP710: footprint Library:TP_0.5mm -> lib:TP_0.5
Connections:
- net GND: now also D3.2
- net NRST: now also D3.1
