File: PCB/RCC_BOOT_RST_DEBUG.kicad_sch (KiCad schematic)
At the start: 38 parts, among them J701 FTSH-107-01-L-DV-K-A, U301 STM32MP157FABx, U701 HSP051-4M10, U702 HSP051-4M10, Y701 ECS-2520MVQ-240

Commit message: PCB_UPDATE
Parts:
- removed R704, R705, R707, R708: 0, Resistor_SMD:R_0402_1005Metric, symbol Device:R
- added D5: MSP3V3-M3/89A, Diode_SMD:D_MicroSMP_KA, symbol PTVS3V3S1UR:PTVS3V3S1UR
Connections:
- net GND: now also D5.2
- net VDD: now also U301.N1 (PDR_ON_CORE), U301.N2 (PDR_ON), D5.1

Commit message: PCB_UPDATE
Parts:
- removed D3: MSP3V3-M3/89A, Diode_SMD:D_MicroSMP_KA, symbol PTVS3V3S1UR:PTVS3V3S1UR
Other:
- moved on the sheet: C701
