File: PCB/RCC_BOOT_RST_DEBUG.kicad_sch (KiCad schematic)
At the start: 30 parts, among them J2 FTSH-107-01-L-DV-K-A, U4 STM32MP157FABx, U8 HSP051-4M10, U9 HSP051-4M10, Y2 ECS-2520MVQ-240

Commit message: PCB_UPDATE
Parts:
- C112, C113, C115: LCSC Part # (none) -> C15195; P/N GRM155R71C103KA01J -> (none); REC P/N (none) -> GRM155R71C103KA01J
- C114, C116: LCSC Part # (none) -> C88896
- R58, R59, R60, R61, R62, R63, R64, R65: LCSC Part # (none) -> C25744
- R66: LCSC Part # (none) -> C17168
- R67: LCSC Part # (none) -> C11702
- R68: LCSC Part # (none) -> C25077
- R69: LCSC Part # (none) -> C25076
- U4: LCSC Part # (none) -> C1236734
- U8, U9: LCSC Part # (none) -> C1973641; P/N HSP051-4M10 -> (none); REC P/N (none) -> HSP051-4M10
- Y2: P/N ECS-2520MVQ-240-BS-TR -> (none); REC P/N (none) -> ECS-2520MVQ-240-BS-TR

Commit message: UPDATE
Other:
- moved on the sheet: C112, R58, S5

Commit message: UPDATE
Parts:
- renumbered C112 to C701, C113 to C702, C114 to C703, C115 to C704, C116 to C705, J2 to J701, R58 to R701, R59 to R702, R60 to R703, R61 to R704, R62 to R705, R63 to R706, R64 to R707, R65 to R708, R66 to R709, R67 to R710, R68 to R711, R69 to R712, S5 to S701, TP29 to TP701, TP21 to TP702, TP25 to TP703, TP22 to TP704, TP26 to TP705, TP27 to TP706, TP30 to TP707, U8 to U702, U9 to U703, Y2 to Y701

Commit message: UPDATE
Parts:
- removed S701: EVQ-9P701P, lib:SW_EVQ-9P701P, symbol EVQ-9P701P:EVQ-9P701P
- added S1: B3U-3000P, lib:SW_B3U-3000P, symbol B3U-3000P:B3U-3000P
Connections:
- net GND: now also S1.2
- net NRST: now also S1.1
