File: PCB/DDR.kicad_sch (KiCad schematic)
At the start: 65 parts, among them U301 STM32MP157FABx, U401 MT41K256M16TW-107_P

Commit message: PCB_UPDATE
Parts:
- TP401, TP402, TP403: footprint Library:TP_0.5mm -> lib:TP_0.5
Changed lines of the file:
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@@
 		(polyline
 			(pts
-				(xy 194.31 35.56) (xy 214.63 35.56) (xy 214.63 64.77) (xy 194.31 64.77)
+				(xy 167.64 140.97) (xy 167.64 157.48) (xy 175.26 157.48) (xy 175.26 140.97)
 			)
 			(stroke
@@
 		(polyline
 			(pts
-				(xy 294.9575 109.22) (xy 309.5625 109.22) (xy 309.5625 123.19) (xy 294.9575 123.19)
+				(xy 281.94 109.22) (xy 293.37 109.22) (xy 293.37 167.64) (xy 281.305 167.64)
 			)
 			(stroke
@@
 		(polyline
 			(pts
-				(xy 281.94 109.22) (xy 293.37 109.22) (xy 293.37 167.64) (xy 281.305 167.64)
+				(xy 194.31 35.56) (xy 214.63 35.56) (xy 214.63 64.77) (xy 194.31 64.77)
 			)
 			(stroke
@@
 		(polyline
 			(pts
-				(xy 167.64 140.97) (xy 167.64 157.48) (xy 175.26 157.48) (xy 175.26 140.97)
+				(xy 172.72 66.04) (xy 214.3125 66.04) (xy 214.3125 72.39) (xy 172.72 72.39)
 			)
 			(stroke
@@
 		(polyline
 			(pts
-				(xy 172.72 66.04) (xy 214.3125 66.04) (xy 214.3125 72.39) (xy 172.72 72.39)
+				(xy 294.9575 109.22) (xy 309.5625 109.22) (xy 309.5625 123.19) (xy 294.9575 123.19)
 			)
 			(stroke
@@
 			)
 		)
-		(property "Footprint" "Library:TP_0.5mm"
+		(property "Footprint" "lib:TP_0.5"
 			(at 168.91 148.59 0)
 			(effects
@@
 			)
 		)
-		(property "Footprint" "Library:TP_0.5mm"
+		(property "Footprint" "lib:TP_0.5"
 			(at 162.56 148.59 0)
 			(effects
@@
 			)
 		)
-		(property "Footprint" "Library:TP_0.5mm"
+		(property "Footprint" "lib:TP_0.5"
 			(at 156.21 148.59 0)
 			(effects
