File: PCB/DDR.kicad_sch (KiCad schematic)
At the start: 63 parts, among them U4 STM32MP157FABx, U5 MT41K256M16TW-107_P

Commit message: update
Parts:
- removed R37: 56, Resistor_SMD:R_0402_1005Metric, symbol Device:R
Connections:
- net DDR_A15: no longer names the net of U4.L16 (DDR_A15)
- net DDR_A15: no longer U5.M7 (A15)
- no-connect marks 3 -> 5
Changed lines of the file:
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@@
 	)
 	(junction
-		(at 336.55 149.86)
-		(diameter 0)
-		(color 0 0 0 0)
-	)
-	(junction
 		(at 267.97 58.42)
 		(diameter 0)
@@
 	)
 	(no_connect
+		(at 146.05 110.49)
+	)
+	(no_connect
+		(at 215.9 132.08)
+	)
+	(no_connect
 		(at 146.05 148.59)
 	)
@@
 	(wire
 		(pts
-			(xy 336.55 146.05) (xy 336.55 149.86)
+			(xy 336.55 146.05) (xy 336.55 152.4)
 		)
 		(stroke
@@
 	(wire
 		(pts
-			(xy 331.47 149.86) (xy 336.55 149.86)
-		)
-		(stroke
-			(width 0)
-			(type default)
-		)
-	)
-	(wire
-		(pts
 			(xy 269.24 226.06) (xy 269.24 228.6)
 		)
@@
 	(wire
 		(pts
-			(xy 201.93 132.08) (xy 215.9 132.08)
-		)
-		(stroke
-			(width 0)
-			(type default)
-		)
-	)
-	(wire
-		(pts
 			(xy 266.7 81.28) (xy 271.78 81.28)
 		)
@@
 	(wire
 		(pts
-			(xy 336.55 149.86) (xy 336.55 152.4)
-		)
-		(stroke
-			(width 0)
-			(type default)
-		)
-	)
-	(wire
-		(pts
 			(xy 353.06 118.11) (xy 349.25 118.11)
 		)
@@
 	(wire
 		(pts
-			(xy 318.77 149.86) (xy 323.85 149.86)
-		)
-		(stroke
-			(width 0)
-			(type default)
-		)
-	)
-	(wire
-		(pts
 			(xy 267.97 50.8) (xy 267.97 53.34)
 		)
@@
 		)
 	)
-	(label "DDR_A15"
-		(at 201.93 132.08 0)
-		(effects
-			(font
-				(size 1.27 1.27)
-			)
-			(justify left bottom)
-		)
-	)
 	(label "DDR_DQ10"
 		(at 63.5 123.19 180)
@@
 		)
 	)
-	(label "DDR_A15"
-		(at 146.05 110.49 0)
-		(effects
-			(font
-				(size 1.27 1.27)
-			)
-			(justify left bottom)
-		)
-	)
 	(label "DDR_ODT"
 		(at 318.77 170.18 180)
@@
 		)
 	)
-	(label "DDR_A15"
-		(at 318.77 149.86 180)
-		(effects
-			(font
-				(size 1.27 1.27)
-			)
-			(justify right bottom)
-		)
-	)
 	(label "DDR_A6"
 		(at 146.05 87.63 0)
@@
 					(unit 1)
 				)
-			)
-		)
-	)
-	(symbol
-		(lib_id "Device:R")
-		(at 327.66 149.86 90)
-		(unit 1)
-		(exclude_from_sim no)
-		(in_bom yes)
-		(on_board yes)
-		(dnp no)
-		(property "Reference" "R37"
-			(at 323.342 147.828 90)
-			(effects
-				(font
-					(size 1.27 1.27)
-				)
-			)
-		)
-		(property "Value" "56"
-			(at 331.724 148.844 90)
-			(effects
-				(font
-					(size 1.27 1.27)
-				)
-			)
-		)
-		(property "Footprint" "Resistor_SMD:R_0402_1005Metric"
-			(at 327.66 151.638 90)
-			(effects
-				(font
-					(size 1.27 1.27)
-				)
-				(hide yes)
-			)
-		)
-		(property "Datasheet" "~"
-			(at 327.66 149.86 0)
-			(effects
-				(font
-					(size 1.27 1.27)
-				)
-				(hide yes)
-			)
-		)
-		(property "Description" "Resistor"
-			(at 327.66 149.86 0)
-			(effects
-				(font
-					(size 1.27 1.27)
-				)
-				(hide yes)
-			)
-		)
-		(property "Mouser P/N" ""
-			(at 327.66 149.86 0)
-			(effects
-				(font
-					(size 1.27 1.27)
-				)
-				(hide yes)
-			)
-		)
-		(pin "1"
-		)
-		(pin "2"
-		)
-		(instances
-			(project "MPU_MOD"
-				(path "/65890f61-d586-475b-928a-b635a5e4e59e/69214b2b-0971-43f8-ac76-9e3bbab8a034"
-					(reference "R37")
-					(unit 1)
-				)
