File: PCB/DDR.kicad_sch (KiCad schematic)
At the start: 62 parts, among them U4 STM32MP157FABx, U5 MT41K256M16TW-107_P

Commit message: PCB_UPDATE
Parts:
- C1, C101, C102, C104, C105, C106, C107, C108, C2, C3, C79, C80, C81, C83, C84, C85, C86, C87, C88, C89, C90, C91, C92, C93, C94, C95, C96, C98, C99: LCSC Part # (none) -> C307331; P/N GRM155R61E104KA87J -> (none); REC P/N (none) -> GRM155R61E104KA87J
- C100, C103: LCSC Part # (none) -> C96446; P/N GRT188R61A106KE13D -> (none); REC P/N (none) -> GRT188R61A106KE13D
- R17, R18: LCSC Part # (none) -> C25094
- R19: LCSC Part # (none) -> C25076
- R20, R21: LCSC Part # (none) -> C25744
- R22, R23, R24, R25, R26, R27, R28, R29, R30, R31, R32, R33, R34, R35, R36, R38, R39, R40, R41, R42, R43, R44, R45, R46: LCSC Part # (none) -> C25127
- U4: LCSC Part # (none) -> C1236734
- U5: LCSC Part # (none) -> C253882; P/N MT41K256M16TW-107:P -> (none); REC P/N (none) -> MT41K256M16TW-107:P

Commit message: UPDATE
Parts:
- renumbered C79 to C401, C3 to C402, C2 to C403, C83 to C404, C84 to C405, C105 to C406, C1 to C407, C80 to C408, C81 to C409, C85 to C410, C86 to C411, C87 to C412, C88 to C413, C89 to C414, C90 to C415, C91 to C416, C92 to C417, C93 to C418, C94 to C419, C95 to C420, C96 to C421, C98 to C422, C99 to C423, C100 to C424, C101 to C425, C102 to C426, C103 to C427, C104 to C428, C106 to C429, C107 to C430, C108 to C431, R17 to R401, R18 to R402, R19 to R403, R20 to R404, R21 to R405, R22 to R406, R23 to R407, R24 to R408, R25 to R409, R26 to R410, R27 to R411, R28 to R412, R29 to R413, R30 to R414, R31 to R415, R32 to R416, R33 to R417, R34 to R418, R35 to R419, R36 to R420, R38 to R421, R39 to R422, R40 to R423, R41 to R424, R42 to R425, R43 to R426, R44 to R427, R45 to R428, R46 to R429, U5 to U402
