File: PCB/WIFI_BLE.kicad_sch (KiCad schematic)
At the start: 25 parts, among them J901 73412-0110, U901 LBEE5PK2AE-771

Commit message: PCB_UPDATE
Parts:
- TP901, TP902, TP903, TP904, TP905, TP906, TP907, TP908: footprint Library:TP_0.5mm -> lib:TP_0.5
Changed lines of the file:
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@@
 			)
 		)
-		(property "Footprint" "Library:TP_0.5mm"
+		(property "Footprint" "lib:TP_0.5"
 			(at 59.69 130.81 0)
 			(effects
@@
 			)
 		)
-		(property "Footprint" "Library:TP_0.5mm"
+		(property "Footprint" "lib:TP_0.5"
 			(at 106.68 118.11 0)
 			(effects
@@
 			)
 		)
-		(property "Footprint" "Library:TP_0.5mm"
+		(property "Footprint" "lib:TP_0.5"
 			(at 114.3 118.11 0)
 			(effects
@@
 			)
 		)
-		(property "Footprint" "Library:TP_0.5mm"
+		(property "Footprint" "lib:TP_0.5"
 			(at 76.2 130.81 0)
 			(effects
@@
 			)
 		)
-		(property "Footprint" "Library:TP_0.5mm"
+		(property "Footprint" "lib:TP_0.5"
 			(at 69.85 130.81 0)
 			(effects
@@
 			)
 		)
-		(property "Footprint" "Library:TP_0.5mm"
+		(property "Footprint" "lib:TP_0.5"
 			(at 99.06 118.11 0)
 			(effects
@@
 			)
 		)
-		(property "Footprint" "Library:TP_0.5mm"
+		(property "Footprint" "lib:TP_0.5"
 			(at 121.92 118.11 0)
 			(effects
@@
 			)
 		)
-		(property "Footprint" "Library:TP_0.5mm"
+		(property "Footprint" "lib:TP_0.5"
 			(at 64.77 130.81 0)
 			(effects
