File: PCB/WIFI_BLE.kicad_sch (KiCad schematic)
At the start: 26 parts, among them J901 73412-0110, U1 LBEE5KL1YN-814, U901 LBEE5PK2AE-771

Commit message: PCB_UPDATE
Parts:
- removed C901: 4.7uF, lib:C_0402_small, symbol Device:C
- removed C902, C903: 10uF, Capacitor_SMD:C_0603_1608Metric, symbol Device:C
- removed C904, C905: 100nF, lib:C_0402_small, symbol Device:C
- removed J901: 73412-0110, lib:MOLEX_73412-0110, symbol 73412-0110:73412-0110
- removed L901: 1uH, Inductor_SMD:L_Murata_DFE201610P, symbol Device:L
- removed R901, R902, R903: 0, Resistor_SMD:R_0402_1005Metric, symbol Device:R
- removed R904: 22, Resistor_SMD:R_0402_1005Metric, symbol Device:R
- removed R905, R906, R907, R908, R909: 47k, Resistor_SMD:R_0402_1005Metric, symbol Device:R
- removed TP901, TP902, TP903, TP904, TP905, TP906, TP907, TP908: TestPoint, lib:TP_0.5, symbol Connector:TestPoint
- removed U1: LBEE5KL1YN-814, lib:XCVR_LBEE5KL1YN-814, symbol LBEE5KL1YN-814:LBEE5KL1YN-814
- removed U901: LBEE5PK2AE-771, lib:XCVR_LBEE5PK2AE-771, symbol LBEE5PK2AE:LBEE5PK2BC-771
Connections:
- no-connect marks 15 -> 0
