File: PCB/_autosave-MPU_MOD.kicad_pcb (KiCad board)
At the start: 6 copper layers, 43.5 x 90 mm, 257 parts, among them J2 2-1734248-0, J3 USB4510-03-1-A_REVA, J501 MEM2090-00-145-00-A_REVA, J701 FTSH-107-01-L-DV-K-A, Q1 CSD23381F4, U201 STC3115IQT, U203 STPMIC1APQR, U3 BQ24298RTWR, U301 STM32MP157FABx, U401 MT41K256M16TW-107_P, U502 HSP051-4M10, U503 HSP051-4M10, U701 HSP051-4M10, U702 HSP051-4M10, U801 FUSB302BMPX, U802 HSP051-4M10, Y601 NX2012SA-32.768K, Y701 ECS-2520MVQ-240

Commit message: PCB_UPDATE
Parts:
- moved R513 0.08 mm to (79.7, 82.5)
Routing:
- net uSD_DETECT: track 3.49 -> 30.4 mm, vias 1 -> 3
- net SDMMC1_CMD: track 13.8 -> 30.7 mm, vias 3 -> 2
- net SDMMC1_D2: track 18.9 -> 35.0 mm
- net SDMMC1_CK: track 23.6 -> 38.5 mm, vias 3 -> 4
- net SDMMC1_D1: track 26.9 -> 38.7 mm, vias 2 -> 4
- net SDMMC1_D3: track 22.3 -> 32.4 mm, vias 3 -> 4
- net SDMMC1_D0: track 33.6 -> 38.6 mm, vias 1 -> 2
- net Net-(J501-SWITCH): track 13.8 -> 17.7 mm, vias 0 -> 1
