File: PCB/DAC.kicad_sch (KiCad schematic)
At the start: 1 part, among them J1 SJ-43504-SMT-TR

Commit message: PCB_UPDATE
Parts:
- removed J1: SJ-43504-SMT-TR, lib:CUI_SJ-43504-SMT-TR, symbol SJ-43504-SMT-TR:SJ-43504-SMT-TR
