File: PCB/MODULE_CONNECTOR.kicad_sch (KiCad schematic)
At the start: 1 part, among them J4 Conn_02x15_Odd_Even

Commit message: pcb update
Parts:
- removed J4: Conn_02x15_Odd_Even, Connector_PinHeader_2.54mm:PinHeader_2x15_P2.54mm_Horizontal, symbol Connector_Generic:Conn_02x15_Odd_Even
Changed lines of the file:
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@@
 	(generator_version "9.0")
 	(paper "A4")
-	(symbol
-		(lib_id "Connector_Generic:Conn_02x15_Odd_Even")
-		(at 127 80.01 0)
-		(unit 1)
-		(exclude_from_sim no)
-		(in_bom yes)
-		(on_board yes)
-		(dnp no)
-		(fields_autoplaced yes)
-		(property "Reference" "J4"
-			(at 128.27 55.88 0)
-			(effects
-				(font
-					(size 1.27 1.27)
-				)
-			)
-		)
-		(property "Value" "Conn_02x15_Odd_Even"
-			(at 128.27 58.42 0)
-			(effects
-				(font
-					(size 1.27 1.27)
-				)
-			)
-		)
-		(property "Footprint" "Connector_PinHeader_2.54mm:PinHeader_2x15_P2.54mm_Horizontal"
-			(at 127 80.01 0)
-			(effects
-				(font
-					(size 1.27 1.27)
-				)
-				(hide yes)
-			)
-		)
-		(property "Datasheet" "~"
-			(at 127 80.01 0)
-			(effects
-				(font
-					(size 1.27 1.27)
-				)
-				(hide yes)
-			)
-		)
-		(property "Description" "Generic connector, double row, 02x15, odd/even pin numbering scheme (row 1 odd numbers, row 2 even numbers), script generated (kicad-library-utils/schlib/autogen/connector/)"
-			(at 127 80.01 0)
-			(effects
-				(font
-					(size 1.27 1.27)
-				)
-				(hide yes)
-			)
-		)
-		(pin "1"
-		)
-		(pin "5"
-		)
-		(pin "3"
-		)
-		(pin "7"
-		)
-		(pin "18"
-		)
-		(pin "16"
-		)
-		(pin "26"
-		)
-		(pin "29"
-		)
-		(pin "2"
-		)
-		(pin "8"
-		)
-		(pin "9"
-		)
-		(pin "17"
-		)
-		(pin "11"
-		)
-		(pin "4"
-		)
-		(pin "14"
-		)
-		(pin "15"
-		)
-		(pin "25"
-		)
-		(pin "6"
-		)
-		(pin "20"
-		)
-		(pin "27"
-		)
-		(pin "24"
-		)
-		(pin "22"
-		)
-		(pin "30"
-		)
-		(pin "19"
-		)
-		(pin "13"
-		)
-		(pin "21"
-		)
-		(pin "10"
-		)
-		(pin "12"
-		)
-		(pin "23"
-		)
-		(pin "28"
-		)
-		(instances
-			(project ""
-				(path "/65890f61-d586-475b-928a-b635a5e4e59e/ba2dc7bc-21cc-4648-b7c2-5eb24b24edf1"
-					(reference "J4")
-					(unit 1)
-				)
-			)
-		)
-	)
 )
