File: PCB/LCD.kicad_sch (KiCad schematic)
At the start: 13 parts, among them J3 FH12-30S-0.5SH_55_, U1 TPS61042DRBR

Commit message: update
Parts:
- added Q2, Q3, Q4: CSD13380F3, Package_DFN_QFN:Texas_PicoStar_DFN-3_0.69x0.60mm, symbol Transistor_FET:CSD13380F3
- added R10, R12, R13, R37, R6, R7, R8, R9: 4k7, Resistor_SMD:R_0402_1005Metric, symbol Device:R
- added R71: 0, Resistor_SMD:R_0402_1005Metric, symbol Device:R
- added TP13, TP14, TP15, TP23, TP24, TP3: TestPoint, lib:TP_0.5, symbol Connector:TestPoint
Connections:
- net GND: now also Q2.2 (S), Q3.2 (S), Q4.2 (S), R10.1, R13.1, R9.1, TP14.1
- net RESET: now also Q2.3 (D), R8.1, TP15.1
- net TP_INT: now also Q3.1 (G), R10.2, TP23.1
- net TP_RES: now also Q4.3 (D), R37.1, TP24.1
- net  LED_A renamed LED_A
- net  LED_K renamed LED_K
- net +1V8 renamed 1V8
- net 1V8: now also R37.2, R6.2, R7.2, R8.2
- net +2V8 renamed 2V8
- net +3V3 renamed 3V3
- net 3V3: now also R12.2
- net DC_LED_PWM: no longer names the net of U1.5 (CTRL)
- net DC_LED_PWM: now also R71.1
- net TP_SCL renamed I2C1_SCL
- net I2C1_SCL: now also R6.1, TP3.1
- net TP_SDA renamed I2C1_SDA
- net I2C1_SDA: now also R7.1, TP13.1
- new net LCD_BL_PWM: R71.2
- new net LCD_RST: Q2.1 (G), R9.2
- new net LCD_TP_INTR: Q3.3 (D), R12.1
- new net LCD_TP_RST: Q4.1 (G), R13.2
Other:
- note added: "DON`T USE INTERNAL PULL UP OR PD"
- moved on the sheet: C35, C5, C9, D1, L1, R11, R5, U1
