File: PCB/LCD.kicad_sch (KiCad schematic)
At the start: 31 parts, among them J3 FH12-30S-0.5SH_55_, Q2 CSD13380F3, Q3 CSD13380F3, Q4 CSD13380F3, U1 TPS61042DRBR

Commit message: PCB_UPDATE
Parts:
- removed R5: 2, Resistor_SMD:R_0402_1005Metric, symbol Device:R
- C35: LCSC Part # (none) -> C52923; P/N GRM155R61E105KA12D -> (none); REC P/N (none) -> GRM155R61E105KA12D
- C4, C5, C6: value 0.47uF -> 1uF; LCSC Part # (none) -> C52923; REC P/N (none) -> GRM155R61E105KA12D
- C7, C8: LCSC Part # (none) -> C307331
- C9: LCSC Part # (none) -> C23733; P/N GRM155R60J475ME47 -> (none); REC P/N (none) -> GRM155R60J475ME47
- D1: LCSC Part # (none) -> C191023
- J3: LCSC Part # (none) -> C506793
- L1: value L -> 4.7uH; LCSC Part # (none) -> C703083; REC P/N (none) -> DFE322512F-4R7M=P2
- R10, R12, R13, R37, R8, R9: value 4k7 -> 10k; LCSC Part # (none) -> C25744
- R11: value 4.7 -> 6.8; LCSC Part # (none) -> C38373
- R6, R7: value 4k7 -> 3k; LCSC Part # (none) -> C25784
- R71: LCSC Part # (none) -> C17168
- U1: LCSC Part # (none) -> C91304
Connections:
- net at R11.2: now also U1.2 (RS), U1.4 (FB)

Commit message: UPDATE
Other:
- note added: "NEED REVIEW"
- note removed: "DON`T USE INTERNAL PULL UP OR PD"
Changed lines of the file:
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@@
 	(generator_version "9.0")
 	(paper "A4")
-	(text "DON`T USE  INTERNAL PULL UP OR PD "
+	(text "NEED REVIEW"
 		(exclude_from_sim no)
-		(at 227.584 129.286 0)
+		(at 88.646 99.822 0)
 		(effects
 			(font
-				(size 1.27 1.27)
+				(size 2.54 2.54)
+				(color 255 41 58 1)
 			)
 		)

Commit message: UPDATE
Parts:
- renumbered C9 to C1001, C35 to C1002, C7 to C1003, C5 to C1004, C8 to C1005, C4 to C1006, C6 to C1007, D1 to D1001, J3 to J1001, L1 to L1001, Q4 to Q1001, Q3 to Q1002, Q2 to Q1003, R71 to R1001, R13 to R1002, R37 to R1003, R11 to R1004, R12 to R1005, R10 to R1006, R9 to R1007, R8 to R1008, R6 to R1009, R7 to R1010, TP24 to TP1001, TP23 to TP1002, TP15 to TP1003, TP13 to TP1004, TP14 to TP1005, TP3 to TP1006, U1 to U1001

Commit message: UPDATE
Parts:
- removed Q1001, Q1002, Q1003: CSD13380F3, Package_DFN_QFN:Texas_PicoStar_DFN-3_0.69x0.60mm, symbol Transistor_FET:CSD13380F3
- added Q1, Q2, Q3: DMG1012TQ-7, Package_TO_SOT_SMD:SOT-523, symbol Transistor_FET:DMG1012T
Connections:
- net GND: now also Q1.2 (S), Q2.2 (S), Q3.2 (S)
- net LCD_RST: now also Q3.1 (G)
- net LCD_TP_INTR: now also Q2.3 (D)
- net LCD_TP_RST: now also Q1.1 (G)
- net RESET: now also Q3.3 (D)
- net TP_INT: now also Q2.1 (G)
- net TP_RES: now also Q1.3 (D)
