File: PCB/FLASH_SD.kicad_sch (KiCad schematic)
At the start: 13 parts, among them J1 MEM2090-00-145-00-A_REVA, U6 HSP051-4M10, U7 HSP051-4M10

Commit message: PCB_UPDATE
Parts:
- C109: LCSC Part # (none) -> C23733; P/N GRM155R60J475ME47 -> (none); REC P/N (none) -> GRM155R60J475ME47
- D4: LCSC Part # (none) -> C506620
- J1: P/N MEM2090-00-145-00-A -> (none); REC P/N (none) -> MEM2090-00-145-00-A
- R48, R49, R50, R52, R53, R72: LCSC Part # (none) -> C25792
- R51: LCSC Part # (none) -> C25744
- U6, U7: LCSC Part # (none) -> C1973641; P/N HSP051-4M10 -> (none); REC P/N (none) -> HSP051-4M10
