File: PCB/MPU_MOD.kicad_sch (KiCad schematic)
At the start: 2 parts

Commit message: UPDATE
Parts:
- renumbered H3 to H101, H4 to H102
Changed lines of the file:
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@@
 		(on_board yes)
 		(dnp no)
-		(property "Reference" "#PWR0158"
+		(property "Reference" "#PWR0102"
 			(at 78.74 40.64 0)
 			(effects
@@
 			(project "MPU_MOD"
 				(path "/65890f61-d586-475b-928a-b635a5e4e59e"
-					(reference "#PWR0158")
+					(reference "#PWR0102")
 					(unit 1)
 				)
@@
 		(dnp no)
 		(fields_autoplaced yes)
-		(property "Reference" "H3"
+		(property "Reference" "H101"
 			(at 57.15 30.4799 0)
 			(effects
@@
 			(project "MPU_MOD"
 				(path "/65890f61-d586-475b-928a-b635a5e4e59e"
-					(reference "H3")
+					(reference "H101")
 					(unit 1)
 				)
@@
 		(on_board yes)
 		(dnp no)
-		(property "Reference" "#PWR0159"
+		(property "Reference" "#PWR0101"
 			(at 54.61 41.91 0)
 			(effects
@@
 			(project "MPU_MOD"
 				(path "/65890f61-d586-475b-928a-b635a5e4e59e"
-					(reference "#PWR0159")
+					(reference "#PWR0101")
 					(unit 1)
 				)
@@
 		(dnp no)
 		(fields_autoplaced yes)
-		(property "Reference" "H4"
+		(property "Reference" "H102"
 			(at 81.28 29.2099 0)
 			(effects
@@
 			(project "MPU_MOD"
 				(path "/65890f61-d586-475b-928a-b635a5e4e59e"
-					(reference "H4")
+					(reference "H102")
 					(unit 1)
 				)
@@
 			(project "MPU_MOD"
 				(path "/65890f61-d586-475b-928a-b635a5e4e59e"
-					(page "11")
+					(page "9")
 				)
 			)
@@
 			(project "MPU_MOD"
 				(path "/65890f61-d586-475b-928a-b635a5e4e59e"
-					(page "12")
+					(page "10")
 				)
 			)
@@
 			(project "MPU_MOD"
 				(path "/65890f61-d586-475b-928a-b635a5e4e59e"
-					(page "13")
-				)
-			)
+					(page "11")
+				)
+			)
