File: PCB/IO_Perph_Conn.kicad_sch (KiCad schematic)
At the start: 17 parts, among them U4 STM32MP157FABx, Y1 NX2012SA-32.768K

Commit message: update
Connections:
- net uSD_DETECT: now also U4.B3 (PE6)
- net LCD_TP_RST: now reaches U4.V10 (PE10)
- net LCD_BL_PWM: now reaches U4.V9 (PF6)
- net LCD_TP_INTR: now reaches U4.W10 (PG7)
- net LCD_RST: now reaches U4.V8 (PD11)
Changed lines of the file:
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@@
 				)
 			)
-			(table_cell ""
+			(table_cell "LCD_BL_PWM"
 				(exclude_from_sim no)
 				(at 330.2 205.74 0)
@@
 				)
 			)
-			(table_cell ""
+			(table_cell "PF6"
 				(exclude_from_sim no)
 				(at 354.33 205.74 0)
@@
 				)
 			)
-			(table_cell ""
+			(table_cell "V9"
 				(exclude_from_sim no)
 				(at 378.46 205.74 0)
@@
 		)
 	)
-	(global_label "CHRG_STAT"
-		(shape input)
-		(at 162.56 151.13 180)
-		(fields_autoplaced yes)
-		(effects
-			(font
-				(size 1.27 1.27)
-			)
-			(justify right)
-		)
-		(property "Intersheetrefs" "${INTERSHEET_REFS}"
-			(at 149.2334 151.13 0)
-			(effects
-				(font
-					(size 1.27 1.27)
-				)
-				(justify right)
-				(hide yes)
-			)
-		)
-	)
 	(global_label "SDMMC1_D0"
 		(shape input)
@@
 		)
 	)
+	(global_label "LCD_BL_PWM"
+		(shape input)
+		(at 271.78 74.93 0)
+		(fields_autoplaced yes)
+		(effects
+			(font
+				(size 1.27 1.27)
+			)
+			(justify left)
+		)
+		(property "Intersheetrefs" "${INTERSHEET_REFS}"
+			(at 286.7394 74.93 0)
+			(effects
+				(font
+					(size 1.27 1.27)
+				)
+				(justify left)
+				(hide yes)
+			)
+		)
+	)
 	(global_label "SYS_I2C6_SDA"
 		(shape input)
@@
 		)
 	)
-	(global_label "CHRG_OTG_ON"
-		(shape input)
-		(at 162.56 146.05 180)
-		(fields_autoplaced yes)
-		(effects
-			(font
-				(size 1.27 1.27)
-			)
-			(justify right)
-		)
-		(property "Intersheetrefs" "${INTERSHEET_REFS}"
-			(at 146.27 146.05 0)
+	(global_label "uSD_DETECT"
+		(shape input)
+		(at 227.33 90.17 180)
+		(fields_autoplaced yes)
+		(effects
+			(font
+				(size 1.27 1.27)
+			)
+			(justify right)
+		)
+		(property "Intersheetrefs" "${INTERSHEET_REFS}"
+			(at 212.9755 90.17 0)
 			(effects
 				(font
@@
 		)
 	)
+	(global_label "LCD_TP_RST"
+		(shape input)
+		(at 227.33 100.33 180)
+		(fields_autoplaced yes)
+		(effects
+			(font
+				(size 1.27 1.27)
+			)
+			(justify right)
+		)
+		(property "Intersheetrefs" "${INTERSHEET_REFS}"
+			(at 213.1568 100.33 0)
+			(effects
+				(font
+					(size 1.27 1.27)
+				)
+				(justify right)
+				(hide yes)
+			)
+		)
+	)
 	(global_label "SDMMC3_D3"
 		(shape input)
@@
 		)
 	)
-	(global_label "INT_USB_ctrl"
-		(shape input)
-		(at 151.13 196.85 180)
-		(fields_autoplaced yes)
-		(effects
-			(font
-				(size 1.27 1.27)
-			)
-			(justify right)
-		)
-		(property "Intersheetrefs" "${INTERSHEET_REFS}"
-			(at 136.231 196.85 0)
-			(effects
-				(font
-					(size 1.27 1.27)
-				)
-				(justify right)
+	(global_label "LCD_RST"
+		(shape input)
+		(at 162.56 121.92 0)
+		(fields_autoplaced yes)
+		(effects
+			(font
+				(size 1.27 1.27)
+			)
+			(justify left)
+		)
+		(property "Intersheetrefs" "${INTERSHEET_REFS}"
+			(at 173.528 121.92 0)
+			(effects
+				(font
+					(size 1.27 1.27)
+				)
+				(justify left)
 				(hide yes)
 			)
@@
 		)
 	)
-	(global_label "CHRG_NPG"
-		(shape input)
-		(at 162.56 148.59 180)
-		(fields_autoplaced yes)
-		(effects
-			(font
-				(size 1.27 1.27)
-			)
-			(justify right)
-		)
-		(property "Intersheetrefs" "${INTERSHEET_REFS}"
-			(at 149.5962 148.59 0)
-			(effects
-				(font
-					(size 1.27 1.27)
-				)
-				(justify right)
+	(global_label "LCD_TP_INTR"
+		(shape input)
+		(at 271.78 95.25 0)
+		(fields_autoplaced yes)
+		(effects
+			(font
+				(size 1.27 1.27)
+			)
+			(justify left)
+		)
+		(property "Intersheetrefs" "${INTERSHEET_REFS}"
+			(at 286.679 95.25 0)
+			(effects
+				(font
+					(size 1.27 1.27)
+				)
+				(justify left)
 				(hide yes)
 			)
@@
 		)
 	)
-	(global_label "CHRG_OFF"
-		(shape input)
-		(at 162.56 153.67 180)
-		(fields_autoplaced yes)
-		(effects
-			(font
-				(size 1.27 1.27)
-			)
-			(justify right)
-		)
-		(property "Intersheetrefs" "${INTERSHEET_REFS}"
-			(at 149.959 153.67 0)
-			(effects
-				(font
-					(size 1.27 1.27)
-				)
-				(justify right)
-				(hide yes)
-			)
-		)
-	)
-	(global_label "BAT_FUEL_ALARM"
-		(shape input)
-		(at 121.92 153.67 180)
-		(fields_autoplaced yes)
-		(effects
-			(font
-				(size 1.27 1.27)
-			)
-			(justify right)
-		)
-		(property "Intersheetrefs" "${INTERSHEET_REFS}"
-			(at 103.1505 153.67 0)
-			(effects
-				(font
-					(size 1.27 1.27)
-				)
-				(justify right)
-				(hide yes)
-			)
-		)
-	)
 	(global_label "SDMMC1_D1"
 		(shape input)
@@
 		)
 	)
-	(global_label "PMIC_PA0_WKUP_INTR"
-		(shape input)
-		(at 158.75 176.53 180)
-		(fields_autoplaced yes)
-		(effects
-			(font
-				(size 1.27 1.27)
-			)
-			(justify right)
-		)
-		(property "Intersheetrefs" "${INTERSHEET_REFS}"
-			(at 135.2029 176.53 0)
-			(effects
-				(font
-					(size 1.27 1.27)
-				)
-				(justify right)
-				(hide yes)
-			)
-		)
-	)
 	(global_label "SPI5_MOSI"
 		(shape input)
@@
 				(hide yes)
 			)
-		)
-	)
-	(global_label "BAT_FUEL_RSDTIO"
-		(shape input)
-		(at 121.92 156.21 180)
-		(fields_autoplaced yes)
-		(effects
-			(font
-				(size 1.27 1.27)
-			)
-			(justify right)
-		)
-		(property "Intersheetrefs" "${INTERSHEET_REFS}"
-			(at 102.4248 156.21 0)
-			(effects
-				(font
-					(size 1.27 1.27)
-				)
-				(justify right)
-				(hide yes)
-			)

Commit message: PCB_UPDATE
Parts:
- C110, C111: LCSC Part # (none) -> C88896
- D5, D6: LCSC Part # (none) -> C130723
- R3, R4: LCSC Part # (none) -> C25792
- R56, R57: value 4k7 -> 3k; LCSC Part # (none) -> C25784
- U4: LCSC Part # (none) -> C1236734
- Y1: LCSC Part # (none) -> C891748

Commit message: UPDATE
Connections:
- net uSD_DETECT: now also U4.A5 (PE3); no longer U4.B3 (PE6)
- no-connect marks 0 -> 35
Other:
- note added: "Need R calc"
Changed lines of the file:
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@@
 		(comment 1 "Author: Mykola Grodskyi")
 	)
+	(text "Need R calc\n"
+		(exclude_from_sim no)
+		(at 58.42 71.882 0)
+		(effects
+			(font
+				(size 1.27 1.27)
+			)
+		)
+	)
 	(junction
 		(at 78.74 83.82)
@@
 		(color 0 0 0 0)
 	)
+	(no_connect
+		(at 105.41 106.68)
+	)
+	(no_connect
+		(at 271.78 85.09)
+	)
+	(no_connect
+		(at 162.56 129.54)
+	)
+	(no_connect
+		(at 162.56 101.6)
+	)
+	(no_connect
+		(at 162.56 116.84)
+	)
+	(no_connect
+		(at 162.56 68.58)
+	)
+	(no_connect
+		(at 105.41 66.04)
+	)
+	(no_connect
+		(at 105.41 58.42)
+	)
+	(no_connect
+		(at 105.41 76.2)
+	)
+	(no_connect
+		(at 271.78 100.33)
+	)
+	(no_connect
+		(at 227.33 85.09)
+	)
+	(no_connect
+		(at 227.33 90.17)
+	)
+	(no_connect
+		(at 271.78 92.71)
+	)
+	(no_connect
+		(at 162.56 55.88)
+	)
+	(no_connect
+		(at 162.56 114.3)
+	)
+	(no_connect
+		(at 162.56 50.8)
+	)
+	(no_connect
+		(at 162.56 132.08)
+	)
+	(no_connect
+		(at 227.33 102.87)
+	)
+	(no_connect
+		(at 227.33 105.41)
+	)
+	(no_connect
+		(at 227.33 87.63)
+	)
+	(no_connect
+		(at 162.56 119.38)
+	)
+	(no_connect
+		(at 105.41 96.52)
+	)
+	(no_connect
+		(at 162.56 109.22)
+	)
+	(no_connect
+		(at 271.78 107.95)
+	)
+	(no_connect
+		(at 105.41 119.38)
+	)
+	(no_connect
+		(at 271.78 97.79)
+	)
+	(no_connect
+		(at 162.56 66.04)
+	)
+	(no_connect
+		(at 105.41 93.98)
+	)
+	(no_connect
+		(at 227.33 97.79)
+	)
+	(no_connect
+		(at 162.56 58.42)
+	)
+	(no_connect
+		(at 227.33 107.95)
+	)
+	(no_connect
+		(at 271.78 87.63)
+	)
+	(no_connect
+		(at 227.33 80.01)
+	)
+	(no_connect
+		(at 271.78 113.03)
+	)
+	(no_connect
+		(at 271.78 102.87)
+	)
 	(wire
 		(pts
@@
 	(wire
 		(pts
-			(xy 97.79 50.8) (xy 105.41 50.8)
-		)
-		(stroke
-			(width 0)
-			(type default)
-		)
-	)
-	(wire
-		(pts
 			(xy 58.42 86.36) (xy 105.41 86.36)
 		)
@@
 			(font
 				(size 1.27 1.27)
+				(color 42 55 255 1)
 			)
 			(justify right)
@@
 			(font
 				(size 1.27 1.27)
+				(color 42 55 255 1)
 			)
 			(justify right)
@@
 			(font
 				(size 1.27 1.27)
+				(color 42 55 255 1)
 			)
 			(justify right)
@@
 			(font
 				(size 1.27 1.27)
+				(color 42 55 255 1)
 			)
 			(justify left)
@@
 			(font
 				(size 1.27 1.27)
+				(color 42 55 255 1)
 			)
 			(justify right)
@@
 			(font
 				(size 1.27 1.27)
+				(color 42 55 255 1)
 			)
 			(justify right)
@@
 	(global_label "uSD_DETECT"
 		(shape input)
-		(at 227.33 90.17 180)
+		(at 227.33 82.55 180)
 		(fields_autoplaced yes)
 		(effects
@@
 		)
 		(property "Intersheetrefs" "${INTERSHEET_REFS}"
-			(at 212.9755 90.17 0)
+			(at 212.9755 82.55 0)
 			(effects
 				(font
@@
 			(font
 				(size 1.27 1.27)
+				(color 42 55 255 1)
 			)
 			(justify right)
@@
 			(font
 				(size 1.27 1.27)
+				(color 42 55 255 1)
 			)
 			(justify right)
@@
 			(font
 				(size 1.27 1.27)
+				(color 42 55 255 1)
 			)
 			(justify left)
@@
 			(font
 				(size 1.27 1.27)
+				(color 42 55 255 1)
 			)
 			(justify left)
@@
 		)
 	)
-	(global_label "uSD_DETECT"
-		(shape input)
-		(at 80.01 106.68 180)
-		(fields_autoplaced yes)
-		(effects
-			(font
-				(size 1.27 1.27)
-			)
-			(justify right)
-		)
-		(property "Intersheetrefs" "${INTERSHEET_REFS}"
-			(at 65.6555 106.68 0)
-			(effects
-				(font
-					(size 1.27 1.27)
-				)
-				(justify right)
-				(hide yes)
-			)
-		)
-	)
 	(global_label "UART7_RX_STM"
 		(shape input)
@@
 			(font
 				(size 1.27 1.27)
+				(color 42 55 255 1)
 			)
 			(justify right)
@@
 			(font
 				(size 1.27 1.27)
+				(color 42 55 255 1)
 			)
 			(justify left)
@@
 	(global_label "PMIC_PA0_WKUP_INTR"
 		(shape input)
-		(at 97.79 50.8 180)
+		(at 105.41 50.8 180)
 		(fields_autoplaced yes)
 		(effects
@@
 		)
 		(property "Intersheetrefs" "${INTERSHEET_REFS}"
-			(at 74.2429 50.8 0)
+			(at 81.8629 50.8 0)
 			(effects
 				(font
@@
 			(font
 				(size 1.27 1.27)
+				(color 42 55 255 1)
 			)
 			(justify right)
@@
 			(font
 				(size 1.27 1.27)
+				(color 42 55 255 1)
 			)
 			(justify right)
@@
 			(font
 				(size 1.27 1.27)
+				(color 42 55 255 1)
 			)
 			(justify left)
@@
 			(font
 				(size 1.27 1.27)
+				(color 42 55 255 1)
 			)
 			(justify right)
@@
 			(font
 				(size 1.27 1.27)
+				(color 42 55 255 1)
 			)
 			(justify right)
@@
 			(font
 				(size 1.27 1.27)
+				(color 42 55 255 1)
 			)
 			(justify right)
@@
 			(font
 				(size 1.27 1.27)
+				(color 42 55 255 1)
 			)
 			(justify right)
@@
 			(font
 				(size 1.27 1.27)
+				(color 42 55 255 1)
 			)
 			(justify right)
@@
 			(font
 				(size 1.27 1.27)
+				(color 42 55 255 1)
 			)
 			(justify right)
@@
 			(font
 				(size 1.27 1.27)
+				(color 42 55 255 1)
 			)
 			(justify right)
@@
 			(font
 				(size 1.27 1.27)
+				(color 42 55 255 1)
 			)
 			(justify left)
@@
 			(font
 				(size 1.27 1.27)
+				(color 42 55 255 1)
 			)
 			(justify left)
@@
 			(font
 				(size 1.27 1.27)
+				(color 42 55 255 1)
 			)
 			(justify right)
@@
 			(font
 				(size 1.27 1.27)
+				(color 42 55 255 1)
 			)
 			(justify right)
@@
 			(font
 				(size 1.27 1.27)
+				(color 42 55 255 1)
 			)
 			(justify right)
@@
 			(font
 				(size 1.27 1.27)
+				(color 42 55 255 1)
 			)
 			(justify right)
@@
 			(font
 				(size 1.27 1.27)
+				(color 42 55 255 1)
 			)
 			(justify right)
