File: PCB/IO_Perph_Conn.kicad_sch (KiCad schematic)
At the start: 17 parts, among them U4 STM32MP157FABx, Y601 NX2012SA-32.768K

Commit message: UPDATE
Parts:
- added J2: Conn_02x06_Odd_Even, Connector_PinHeader_1.00mm:PinHeader_2x06_P1.00mm_Vertical_SMD, symbol Connector_Generic:Conn_02x06_Odd_Even
Connections:
- net MOD_TIM1_CH1_OUT: now reaches U4.W7 (PE9)
- no-connect marks 28 -> 27
