File: PCB/WIFI.kicad_sch (KiCad schematic)
At the start: 17 parts, among them U2 MAYA-W166-00B

Commit message: UPDATE
Parts:
- renumbered C82 to C901, C97 to C902, C36 to C903, C37 to C904, R82 to R901, R81 to R902, R80 to R903, R79 to R904, R78 to R905, R14 to R906, R77 to R907, R76 to R908, R75 to R909, R74 to R910, R73 to R911, R5 to R912, U2 to U901
Changed lines of the file:
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@@
 		(on_board yes)
 		(dnp no)
-		(property "Reference" "#PWR0169"
+		(property "Reference" "#PWR0904"
 			(at 217.17 69.85 0)
 			(effects
@@
 			(project "MPU_MOD"
 				(path "/65890f61-d586-475b-928a-b635a5e4e59e/4988eac5-6207-4695-88c2-59584fd8c847"
-					(reference "#PWR0169")
+					(reference "#PWR0904")
 					(unit 1)
 				)
@@
 		(dnp no)
 		(fields_autoplaced yes)
-		(property "Reference" "R14"
+		(property "Reference" "R906"
 			(at 71.12 92.7099 0)
 			(effects
@@
 			(project "MPU_MOD"
 				(path "/65890f61-d586-475b-928a-b635a5e4e59e/4988eac5-6207-4695-88c2-59584fd8c847"
-					(reference "R14")
+					(reference "R906")
 					(unit 1)
 				)
@@
 		(on_board yes)
 		(dnp no)
-		(property "Reference" "R82"
+		(property "Reference" "R901"
 			(at 36.83 95.2501 0)
 			(effects
@@
 			(project "MPU_MOD"
 				(path "/65890f61-d586-475b-928a-b635a5e4e59e/4988eac5-6207-4695-88c2-59584fd8c847"
-					(reference "R82")
+					(reference "R901")
 					(unit 1)
 				)
@@
 		(dnp no)
 		(fields_autoplaced yes)
-		(property "Reference" "R81"
+		(property "Reference" "R902"
 			(at 40.64 63.4999 0)
 			(effects
@@
 			(project "MPU_MOD"
 				(path "/65890f61-d586-475b-928a-b635a5e4e59e/4988eac5-6207-4695-88c2-59584fd8c847"
-					(reference "R81")
+					(reference "R902")
 					(unit 1)
 				)
@@
 		(dnp no)
 		(fields_autoplaced yes)
-		(property "Reference" "R79"
+		(property "Reference" "R904"
 			(at 53.34 92.7099 0)
 			(effects
@@
 			(project "MPU_MOD"
 				(path "/65890f61-d586-475b-928a-b635a5e4e59e/4988eac5-6207-4695-88c2-59584fd8c847"
-					(reference "R79")
+					(reference "R904")
 					(unit 1)
 				)
@@
 		(on_board yes)
 		(dnp no)
-		(property "Reference" "#PWR0170"
+		(property "Reference" "#PWR0907"
 			(at 229.87 69.85 0)
 			(effects
@@
 			(project "MPU_MOD"
 				(path "/65890f61-d586-475b-928a-b635a5e4e59e/4988eac5-6207-4695-88c2-59584fd8c847"
-					(reference "#PWR0170")
+					(reference "#PWR0907")
 					(unit 1)
 				)
@@
 		(on_board yes)
 		(dnp no)
-		(property "Reference" "C36"
+		(property "Reference" "C903"
 			(at 234.442 76.2 90)
 			(effects
@@
 			(project "MPU_MOD"
 				(path "/65890f61-d586-475b-928a-b635a5e4e59e/4988eac5-6207-4695-88c2-59584fd8c847"
-					(reference "C36")
+					(reference "C903")
 					(unit 1)
 				)
@@
 		(on_board yes)
 		(dnp no)
-		(property "Reference" "C37"
+		(property "Reference" "C904"
 			(at 235.712 58.42 90)
 			(effects
@@
 			(project "MPU_MOD"
 				(path "/65890f61-d586-475b-928a-b635a5e4e59e/4988eac5-6207-4695-88c2-59584fd8c847"
-					(reference "C37")
+					(reference "C904")
 					(unit 1)
 				)
@@
 		(dnp no)
 		(fields_autoplaced yes)
-		(property "Reference" "R78"
+		(property "Reference" "R905"
 			(at 62.23 92.7099 0)
 			(effects
@@
 			(project "MPU_MOD"
 				(path "/65890f61-d586-475b-928a-b635a5e4e59e/4988eac5-6207-4695-88c2-59584fd8c847"
-					(reference "R78")
+					(reference "R905")
 					(unit 1)
 				)
@@
 		(dnp no)
 		(fields_autoplaced yes)
-		(property "Reference" "U2"
+		(property "Reference" "U901"
 			(at 255.27 85.09 0)
 			(effects
@@
 			(project ""
 				(path "/65890f61-d586-475b-928a-b635a5e4e59e/4988eac5-6207-4695-88c2-59584fd8c847"
-					(reference "U2")
+					(reference "U901")
 					(unit 2)
 				)
@@
 		(on_board yes)
 		(dnp no)
-		(property "Reference" "R5"
+		(property "Reference" "R912"
 			(at 78.232 110.744 90)
 			(effects
@@
 			(project "MPU_MOD"
 				(path "/65890f61-d586-475b-928a-b635a5e4e59e/4988eac5-6207-4695-88c2-59584fd8c847"
-					(reference "R5")
+					(reference "R912")
 					(unit 1)
 				)
@@
 		(on_board yes)
 		(dnp no)
-		(property "Reference" "#PWR0171"
+		(property "Reference" "#PWR0903"
 			(at 187.96 138.43 0)
 			(effects
@@
 			(project "MPU_MOD"
 				(path "/65890f61-d586-475b-928a-b635a5e4e59e/4988eac5-6207-4695-88c2-59584fd8c847"
-					(reference "#PWR0171")
+					(reference "#PWR0903")
 					(unit 1)
 				)
@@
 		(on_board yes)
 		(dnp no)
-		(property "Reference" "#PWR0167"
+		(property "Reference" "#PWR0906"
 			(at 228.6 87.63 0)
 			(effects
@@
 			(project "MPU_MOD"
 				(path "/65890f61-d586-475b-928a-b635a5e4e59e/4988eac5-6207-4695-88c2-59584fd8c847"
-					(reference "#PWR0167")
+					(reference "#PWR0906")
 					(unit 1)
 				)
@@
 		(dnp no)
 		(fields_autoplaced yes)
-		(property "Reference" "#PWR0164"
+		(property "Reference" "#PWR0909"
 			(at 241.3 73.66 0)
 			(effects
@@
 			(project "MPU_MOD"
 				(path "/65890f61-d586-475b-928a-b635a5e4e59e/4988eac5-6207-4695-88c2-59584fd8c847"
-					(reference "#PWR0164")
+					(reference "#PWR0909")
 					(unit 1)
 				)
@@
 		(on_board yes)
 		(dnp no)
-		(property "Reference" "#PWR0180"
+		(property "Reference" "#PWR0902"
 			(at 43.18 77.47 0)
 			(effects
@@
 			(project "MPU_MOD"
 				(path "/65890f61-d586-475b-928a-b635a5e4e59e/4988eac5-6207-4695-88c2-59584fd8c847"
-					(reference "#PWR0180")
+					(reference "#PWR0902")
 					(unit 1)
 				)
@@
 		(on_board yes)
 		(dnp no)
-		(property "Reference" "#PWR0168"
+		(property "Reference" "#PWR0905"
 			(at 217.17 87.63 0)
 			(effects
@@
 			(project "MPU_MOD"
 				(path "/65890f61-d586-475b-928a-b635a5e4e59e/4988eac5-6207-4695-88c2-59584fd8c847"
-					(reference "#PWR0168")
+					(reference "#PWR0905")
 					(unit 1)
 				)
@@
 		(on_board yes)
 		(dnp no)
-		(property "Reference" "C82"
+		(property "Reference" "C901"
 			(at 221.742 57.404 0)
 			(effects
@@
 			(project "MPU_MOD"
 				(path "/65890f61-d586-475b-928a-b635a5e4e59e/4988eac5-6207-4695-88c2-59584fd8c847"
-					(reference "C82")
+					(reference "C901")
 					(unit 1)
 				)
@@
 		(dnp no)
 		(fields_autoplaced yes)
-		(property "Reference" "#PWR0179"
+		(property "Reference" "#PWR0901"
 			(at 35.56 87.63 0)
 			(effects
@@
 			(project "MPU_MOD"
 				(path "/65890f61-d586-475b-928a-b635a5e4e59e/4988eac5-6207-4695-88c2-59584fd8c847"
-					(reference "#PWR0179")
+					(reference "#PWR0901")
 					(unit 1)
 				)
@@
 		(on_board yes)
 		(dnp no)
-		(property "Reference" "R73"
+		(property "Reference" "R911"
 			(at 78.232 108.204 90)
 			(effects
@@
 			(project "MPU_MOD"
 				(path "/65890f61-d586-475b-928a-b635a5e4e59e/4988eac5-6207-4695-88c2-59584fd8c847"
-					(reference "R73")
+					(reference "R911")
 					(unit 1)
 				)
@@
 		(on_board yes)
 		(dnp no)
-		(property "Reference" "R74"
+		(property "Reference" "R910"
 			(at 78.232 105.664 90)
 			(effects
@@
 			(project "MPU_MOD"
 				(path "/65890f61-d586-475b-928a-b635a5e4e59e/4988eac5-6207-4695-88c2-59584fd8c847"
-					(reference "R74")
+					(reference "R910")
 					(unit 1)
 				)
@@
 		(on_board yes)
 		(dnp no)
-		(property "Reference" "R77"
+		(property "Reference" "R907"
 			(at 78.232 98.044 90)
 			(effects
@@
 			(project "MPU_MOD"
 				(path "/65890f61-d586-475b-928a-b635a5e4e59e/4988eac5-6207-4695-88c2-59584fd8c847"
-					(reference "R77")
+					(reference "R907")
 					(unit 1)
 				)
@@
 		(on_board yes)
 		(dnp no)
-		(property "Reference" "C97"
+		(property "Reference" "C902"
 			(at 221.742 75.184 0)
 			(effects
@@
 			(project "MPU_MOD"
 				(path "/65890f61-d586-475b-928a-b635a5e4e59e/4988eac5-6207-4695-88c2-59584fd8c847"
-					(reference "C97")
+					(reference "C902")
 					(unit 1)
 				)
@@
 		(on_board yes)
 		(dnp no)
-		(property "Reference" "R76"
+		(property "Reference" "R908"
 			(at 78.232 100.584 90)
 			(effects
@@
 			(project "MPU_MOD"
 				(path "/65890f61-d586-475b-928a-b635a5e4e59e/4988eac5-6207-4695-88c2-59584fd8c847"
-					(reference "R76")
+					(reference "R908")
 					(unit 1)
 				)
@@
 		(dnp no)
 		(fields_autoplaced yes)
-		(property "Reference" "U2"
+		(property "Reference" "U901"
 			(at 149.86 55.88 0)
 			(effects
@@
 			(project ""
 				(path "/65890f61-d586-475b-928a-b635a5e4e59e/4988eac5-6207-4695-88c2-59584fd8c847"
-					(reference "U2")
+					(reference "U901")
 					(unit 1)
 				)
@@
 		(on_board yes)
 		(dnp no)
-		(property "Reference" "R75"
+		(property "Reference" "R909"
 			(at 78.232 103.124 90)
 			(effects
@@
 			(project "MPU_MOD"
 				(path "/65890f61-d586-475b-928a-b635a5e4e59e/4988eac5-6207-4695-88c2-59584fd8c847"
-					(reference "R75")
+					(reference "R909")
 					(unit 1)
 				)
@@
 		(dnp no)
 		(fields_autoplaced yes)
-		(property "Reference" "R80"
+		(property "Reference" "R903"
 			(at 45.72 92.7099 0)
 			(effects
@@
 			(project "MPU_MOD"
 				(path "/65890f61-d586-475b-928a-b635a5e4e59e/4988eac5-6207-4695-88c2-59584fd8c847"
-					(reference "R80")
+					(reference "R903")
 					(unit 1)
 				)
@@
 		(dnp no)
 		(fields_autoplaced yes)
-		(property "Reference" "#PWR0161"
+		(property "Reference" "#PWR0908"
 			(at 241.3 54.61 0)
 			(effects
@@
 			(project "MPU_MOD"
 				(path "/65890f61-d586-475b-928a-b635a5e4e59e/4988eac5-6207-4695-88c2-59584fd8c847"
-					(reference "#PWR0161")
+					(reference "#PWR0908")
 					(unit 1)
 				)

Commit message: UPDATE
Parts:
- removed C903, C904: 10uF, Capacitor_SMD:C_0603_1608Metric, symbol Device:C
- added C1, C4, C5: 100nF, lib:C_0402_small, symbol Device:C
- added C2, C3: 22uF, Capacitor_SMD:C_0603_1608Metric, symbol Device:C
- added C6, C7: 1uF, lib:C_0402_small, symbol Device:C
- added R1: 100, Resistor_SMD:R_0402_1005Metric, symbol Device:R
Connections:
- net 1V8_WIFI: now also C3.1
- net 3V3: now also C2.1, C4.1, C5.1, C6.2, C7.2
- net GND: now also C1.2, C2.2, C3.2, C4.2, C5.2, C6.1, C7.1
- net I2S3_CK: now also U901.D8 (PCM_CLK/GPIO6)
- net I2S3_SDI: now also U901.E9 (PCM_DIN/GPIO5)
- net I2S3_SDO: now also U901.F9 (PCM_DOUT/GPIO4)
- net I2S3_WS: now also U901.F8 (PCM_SYNC/GPIO7)
- net WIFI_PDn: now also R1.1; no longer U901.J3 (PDN)
- net BT_WAKE_HOST: now reaches U901.E7 (BT_WAKE_HOST/GPIO0)
- net WLAN_WAKE_HOST: now reaches U901.F7 (WLAN_WAKE_HOST/GPIO1)
- net WLAN_RESET: now reaches U901.H7 (WLAN_RESET/JTAG_TCK/GPIO14)
- net BT_RESET: now reaches U901.J7 (BT_RESET/JTAG_TMS/GPIO15)
- net WLAN_DEV_WAKE: now reaches U901.J8 (WLAN_DEV_WAKE/GPIO13)
- net BT_DEV_WAKE: now reaches U901.J9 (BT_DEV_WAKE/GPIO12)
- net WIFI_SLP_CLK: no longer names the net of U901.B1 (SLP_CLK_IN)
- new net: C1.1, R1.2, U901.J3 (PDN)
- no-connect marks 5 -> 9
Other:
- note added: "Conf settings during boot. internal pull-up exist. Don't interfere with it through UART or a pull-down on the input."
- note removed: "Can accept 3V3? 1V8 domain"
- moved on the sheet: C901, U901B

Commit message: UPDATE
Parts:
- removed C5: 100nF, lib:C_0402_small, symbol Device:C
- removed C7: 1uF, lib:C_0402_small, symbol Device:C
