File: LCD_Adapter/LCD_Adapter_HAT/LCD_Adapter.kicad_pcb (KiCad board)
At the start: 4 copper layers, 65 x 56.5 mm, 57 parts, among them J1 Conn_01x10, J2 FH12-30S-0.5SH_55_, J3 RPi_GPIO, J4 1-1734248-5, J5 FH12-30S-0.5SH_55_, J6 2-1734248-0, U1 TLV75801PDBV, U2 TLV75801PDBV, U3 TPS61042DRBR

Commit message: UPDATE
Parts:
- removed C12: 100nF, Capacitor_SMD:C_0402_1005Metric
- removed J1: Conn_01x10, Connector_PinHeader_2.54mm:PinHeader_1x10_P2.54mm_Vertical
- removed J4: 1-1734248-5, lib:TE_1-1734248-5
- removed J5: FH12-30S-0.5SH_55_, lib:HIROSE_FH12-30S-0.5SH_55_
- removed R1: 0, Resistor_SMD:R_0603_1608Metric
- added Q1: 2N7002, Package_TO_SOT_SMD:SOT-23, F.Cu at (191.6, 80.1)
- added Q2: 2N7002, Package_TO_SOT_SMD:SOT-23, F.Cu at (191.6, 84.7)
- added R17: 2k7, Resistor_SMD:R_0603_1608Metric, F.Cu at (202.1, 61.4)
- added R18: 15k, Resistor_SMD:R_0603_1608Metric, F.Cu at (202.1, 63.9)
- added R19: 0, Resistor_SMD:R_0603_1608Metric, F.Cu at (192.1, 66.4)
- added R20: 0, Resistor_SMD:R_0603_1608Metric, F.Cu at (192.1, 68.9)
- added R21: 1k, Resistor_SMD:R_0603_1608Metric, F.Cu at (192.1, 71.4)
- added R22: 1k, Resistor_SMD:R_0603_1608Metric, F.Cu at (192.1, 73.9)
- added R23: 200k, Resistor_SMD:R_0603_1608Metric, F.Cu at (192.1, 76.4)
- added R24: 0, Resistor_SMD:R_0603_1608Metric, F.Cu at (196.1, 61.4)
- added R25: 0, Resistor_SMD:R_0603_1608Metric, F.Cu at (196.1, 63.9)
- added R26: 0, Resistor_SMD:R_0603_1608Metric, F.Cu at (196.1, 66.4)
- added R27: 0, Resistor_SMD:R_0603_1608Metric, F.Cu at (196.1, 68.9)
- added R28: 0, Resistor_SMD:R_0603_1608Metric, F.Cu at (196.1, 71.4)
- added TP15: TestPoint, TestPoint:TestPoint_Pad_D1.0mm, F.Cu at (187.6, 88.4)
- added TP16: TestPoint, TestPoint:TestPoint_Pad_D1.0mm, F.Cu at (187.6, 91.4)
- C10, C11, C9: value 100nF -> 0.47uF; footprint Capacitor_SMD:C_0402_1005Metric -> Capacitor_SMD:C_0603_1608Metric
- R10, R11: value 10k -> 0
- R12: value 39k -> 51k
- R13: value 160k -> 220k
- R14: value 230k -> 220k
- R15: value 100k -> 82k
- R6: value 10k -> 100k
- moved C15 104.3 mm to (176.5, 116.1)
- moved C16 104.0 mm to (176.5, 118.0), turned to 0 degrees
- moved C14 98.1 mm to (176.5, 114.1)
- moved TP6 96.0 mm to (187.6, 85.3)
- moved C13 95.0 mm to (176.5, 112.1), turned to 0 degrees
- moved TP1 93.8 mm to (187.6, 79.2)
- moved TP5 93.1 mm to (187.6, 82.3)
- moved R9 86.6 mm to (170.0, 119.9)
- moved R11 84.1 mm to (192.1, 63.9)
- moved TP4 84.0 mm to (173.6, 118.8)
- moved R3 83.4 mm to (170.0, 112.4)
- moved TP3 83.4 mm to (173.6, 115.7)
- moved R4 82.0 mm to (170.0, 114.9)
- moved C7 80.6 mm to (212.6, 110.6)
- moved C8 80.6 mm to (212.7, 104.3)
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Connections:
- C10 pad 1: +3V3 -> +2V8
- C11 pad 1: +3V3 -> +1V8
- J3 pad 14: unconnected-(J3-GND-Pad14) -> GND
- J3 pad 16: unconnected-(J3-BCM23-Pad16) -> Net-(J3-BCM23)
- J3 pad 18: unconnected-(J3-BCM24-Pad18) -> Net-(J3-BCM24)
- J3 pad 20: unconnected-(J3-GND-Pad20) -> GND
- J3 pad 22: unconnected-(J3-BCM25-Pad22) -> Net-(J3-BCM25)
- J3 pad 25: unconnected-(J3-GND-Pad25) -> GND
- J3 pad 30: unconnected-(J3-GND-Pad30) -> GND
- J3 pad 32: unconnected-(J3-BCM12_PWM0-Pad32) -> Net-(J3-BCM12_PWM0)
- J3 pad 33: unconnected-(J3-BCM13_PWM1-Pad33) -> Net-(J3-BCM13_PWM1)
- J3 pad 34: unconnected-(J3-GND-Pad34) -> GND
- J3 pad 37: unconnected-(J3-BCM26-Pad37) -> Net-(J3-BCM26)
- J3 pad 39: unconnected-(J3-GND-Pad39) -> GND
- J3 pad 6: unconnected-(J3-GND-Pad6) -> GND
- J3 pad 9: unconnected-(J3-GND-Pad9) -> GND
- J6 pad 11: TP_SCL -> Net-(J6-Pad11)
- J6 pad 12: TP_SDA -> Net-(J6-Pad12)
- J6 pad 17: Net-(J6-Pad17) -> TP_INT
- J6 pad 31: TP_SCL -> Net-(J6-Pad11)
- J6 pad 32: TP_SDA -> Net-(J6-Pad12)
- J6 pad 37: Net-(J6-Pad17) -> TP_INT
- R10 pad 1: RESET -> Net-(J3-BCM12_PWM0)
- R10 pad 2: +2V8 -> PWM
- R11 pad 1: GND -> Net-(J3-BCM24)
- R11 pad 2: RESET -> TP_INT
- R12 pad 1: GND -> Net-(R12-Pad1)
- R15 pad 1: GND -> Net-(R15-Pad1)
- R2 pad 1: Net-(J6-Pad20) -> Net-(J3-BCM26)
- R2 pad 2: TP_RES -> TE
- R3 pad 2: RESET -> Net-(Q1-G)
- R5 pad 1: Net-(J6-Pad17) -> Net-(J6-Pad19)
- R5 pad 2: TP_INT -> DC_LED_PWM
- R6 pad 1: TP_RES -> GND
- R6 pad 2: +2V8 -> Net-(Q1-G)
- R7 pad 2: TP_RES -> TP_RES_STM_SIDE
- TP1 pad 1: RPI_TP_SDA -> TP_INT
- TP5 pad 1: RPI_TP_SCL -> TP_RES
- TP6 pad 1: GND -> Net-(Q1-G)
Routing:
- net +2V8: track 99.6 -> 8.30 mm, vias 12 -> 3
- net +1V8: track 98.0 -> 8.26 mm, vias 9 -> 3
- net GND: track 91.8 -> 6.89 mm, vias 106 -> 45
- net  LED_A: track 80.9 -> 1.33 mm, vias 5 -> 3
- net LCM_ID: track 75.3 -> 0.00 mm, vias 1 -> 0
- net  LED_K: track 73.3 -> 2.57 mm, vias 4 -> 2
- net RESET: track 62.7 -> 0.00 mm, vias 2 -> 0
- net TP_INT: track 62.6 -> 0.00 mm, vias 3 -> 0
- net TE: track 60.6 -> 0.00 mm, vias 3 -> 0
- net PWM: track 59.1 -> 0.00 mm, vias 3 -> 0
- net TP_RES: track 57.2 -> 0.00 mm, vias 2 -> 0
- net DC_LED_PWM: track 52.5 -> 1.24 mm
- net /STM2LCD/D1_P: track 35.9 -> 0.00 mm
- net /RPI2LCD/RPI_D0_P: track 35.6 -> 0.00 mm
- net /RPI2LCD/RPI_D0_N: track 35.6 -> 0.00 mm
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- removed copper zone on In2.Cu, net +3V3
- removed copper zone on In1.Cu, net GND
Other:
- board size 65 x 56.5 mm -> 100 x 70 mm
