File: LCD_Adapter/LCD_Adapter_HAT/LCD_Adapter.kicad_pcb (KiCad board)
At the start: 4 copper layers, 100 x 70 mm, 99 parts, among them J1 2-84953-0, J2 FH12-30S-0.5SH_55_, J3 RPi_GPIO, J4 Conn_02x20_Odd_Even, Q1 2N7002, Q2 2N7002, U1 TLV75801PDBV, U2 TLV75801PDBV, U3 TPS61042DRBR, U4 PCA9306DCURG4

Commit message: PCB_UPDATE
Parts:
- removed the C1 at (200.3, 129.7)
- removed the C2 at (201.8, 129.7)
- removed the C3 at (198.1, 124.9)
- removed the C4 at (207.2, 131.4)
- removed the C5 at (203.4, 126.5)
- removed the C6 at (204.9, 126.5)
- removed the C7 at (213.4, 131.1)
- removed the C8 at (213.4, 124.8)
- removed the D1 at (216.5, 131.0)
- removed the L1 at (218.3, 127.7)
- removed the R12 at (198.1, 131.9)
- removed the R13 at (198.1, 130.5)
- removed the R14 at (207.2, 125.7)
- removed the R15 at (207.2, 124.3)
- removed the R16 at (211.4, 126.3)
- removed the TP10 at (206.4, 121.1)
- removed the TP11 at (216.8, 121.1)
- removed the TP12 at (218.9, 121.1)
- removed the TP13 at (214.8, 121.1)
- removed the TP14 at (198.3, 121.2)
- removed the TP7 at (204.4, 121.1)
- removed the TP8 at (200.3, 121.2)
- removed the TP9 at (202.3, 121.1)
- removed the U1 at (197.8, 127.7)
- removed the U2 at (207.4, 128.5)
- removed the U3 at (214.8, 127.8)
- moved TP12 113.8 mm to (105.8, 138.2), turned to 0 degrees
- moved R19 112.5 mm to (107.6, 140.7), turned to 90 degrees
- moved R28 110.3 mm to (110.3, 140.7), turned to 90 degrees
- moved TP13 106.3 mm to (108.8, 135.8), turned to 0 degrees
- moved R10 104.8 mm to (123.4, 140.5)
- moved R2 104.1 mm to (112.7, 140.7), turned to 90 degrees
- moved R16 101.7 mm to (117.2, 134.5), turned to 0 degrees
- moved R20 100.3 mm to (123.4, 142.0)
- moved TP11 99.3 mm to (112.6, 102.3), turned to 0 degrees
- moved TP16 99.1 mm to (88.9, 99.9)
- moved C8 98.5 mm to (119.4, 136.3), turned to 180 degrees
- moved R18 97.3 mm to (129.1, 128.2), turned to 0 degrees
- moved C7 96.0 mm to (119.3, 130.1), turned to 180 degrees
- moved U3 94.4 mm to (120.7, 133.2), turned to 90 degrees
- moved R17 94.0 mm to (136.4, 128.5), turned to 0 degrees
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Connections:
- J4 pad 16: unconnected-(J4-Pin_16-Pad16) -> Net-(J4-Pin_16)
- J4 pad 18: unconnected-(J4-Pin_18-Pad18) -> Net-(J4-Pin_18)
- J4 pad 22: unconnected-(J4-Pin_22-Pad22) -> Net-(J4-Pin_22)
- J4 pad 32: unconnected-(J4-Pin_32-Pad32) -> Net-(J4-Pin_32)
- R10 pad 1: Net-(J3-BCM12_PWM0) -> Net-(J4-Pin_32)
- R19 pad 1: Net-(J3-BCM23) -> Net-(J4-Pin_16)
- R2 pad 1: Net-(J3-BCM26) -> Net-(J4-Pin_22)
- R20 pad 1: Net-(J3-BCM13_PWM1) -> Net-(J4-Pin_32)
- R28 pad 1: Net-(J3-BCM25) -> Net-(J4-Pin_18)
Routing:
- net +1V8: track 8.26 -> 184.5 mm, vias 3 -> 12
- net +2V8: track 8.30 -> 139.8 mm, vias 3 -> 7
- net  LED_A: track 1.33 -> 88.9 mm
- net GND: track 6.89 -> 91.3 mm, vias 45 -> 76
- net  LED_K: track 2.57 -> 80.5 mm, vias 2 -> 3
- net TE: track 0.00 -> 72.2 mm, vias 0 -> 2
- net PWM: track 0.00 -> 68.4 mm, vias 0 -> 2
- net DC_LED_PWM: track 1.24 -> 62.8 mm, vias 1 -> 3
- net LCM_ID: track 0.00 -> 44.3 mm
- net TP_INT: track 0.00 -> 38.6 mm, vias 0 -> 2
- net TP_SCL: track 0.00 -> 38.0 mm
- net RESET: track 0.00 -> 34.5 mm
- net TP_SDA: track 0.00 -> 34.1 mm
- net TP_RES: track 0.00 -> 23.8 mm
- net TP_RES_STM_SIDE: track 0.00 -> 20.5 mm
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- added copper zone on B.Cu, net  LED_A
- added copper zone on In1.Cu, net +1V8
- added copper zone on In1.Cu, net +2V8
- added copper zone on B.Cu, net +3V3
- added copper zone on In1.Cu, net +3V3
- added copper zone on In2.Cu, net GND
- added copper zone on B.Cu, net Net-(D1-A)
- removed copper zone on F.Cu, net  LED_A
- removed copper zone on F.Cu, net +3V3
- removed copper zone on F.Cu, net GND
- removed copper zone on F.Cu, net Net-(D1-A)
Other:
- board size 100 x 70 mm -> 100 x 60 mm
