File: LCD_Adapter/LCD_Adapter_HAT/LCD_Adapter.kicad_sch (KiCad schematic)
At the start: 1 part, among them J3 RPi_GPIO

Commit message: UPDATE
Parts:
- removed J3: RPi_GPIO, lib:RPI_Hat_B+, symbol RPi_Hat:RPi_GPIO
Changed lines of the file:
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@@
-		)
-	)
-	(symbol
-		(lib_id "RPi_Hat:RPi_GPIO")
-		(at 332.74 25.4 0)
-		(unit 1)
-		(exclude_from_sim no)
-		(in_bom yes)
-		(on_board yes)
-		(dnp no)
-		(fields_autoplaced yes)
-		(property "Reference" "J3"
-			(at 351.79 17.78 0)
-			(effects
-				(font
-					(size 1.524 1.524)
-				)
-			)
-		)
-		(property "Value" "RPi_GPIO"
-			(at 351.79 20.32 0)
-			(effects
-				(font
-					(size 1.524 1.524)
-				)
-			)
-		)
-		(property "Footprint" "lib:RPI_Hat_B+"
-			(at 332.74 25.4 0)
-			(effects
-				(font
-					(size 1.524 1.524)
-				)
-			)
-		)
-		(property "Datasheet" ""
-			(at 332.74 25.4 0)
-			(effects
-				(font
-					(size 1.524 1.524)
-				)
-			)
-		)
-		(property "Description" ""
-			(at 332.74 25.4 0)
-			(effects
-				(font
-					(size 1.27 1.27)
-				)
-				(hide yes)
-			)
-		)
-		(pin "9"
-		)
-		(pin "17"
-		)
-		(pin "23"
-		)
-		(pin "27"
-		)
-		(pin "35"
-		)
-		(pin "13"
-		)
-		(pin "21"
-		)
-		(pin "31"
-		)
-		(pin "4"
-		)
-		(pin "6"
-		)
-		(pin "8"
-		)
-		(pin "1"
-		)
-		(pin "7"
-		)
-		(pin "5"
-		)
-		(pin "3"
-		)
-		(pin "11"
-		)
-		(pin "15"
-		)
-		(pin "19"
-		)
-		(pin "25"
-		)
-		(pin "29"
-		)
-		(pin "33"
-		)
-		(pin "37"
-		)
-		(pin "39"
-		)
-		(pin "2"
-		)
-		(pin "28"
-		)
-		(pin "14"
-		)
-		(pin "32"
-		)
-		(pin "36"
-		)
-		(pin "38"
-		)
-		(pin "40"
-		)
-		(pin "16"
-		)
-		(pin "18"
-		)
-		(pin "26"
-		)
-		(pin "24"
-		)
-		(pin "10"
-		)
-		(pin "12"
-		)
-		(pin "20"
-		)
-		(pin "22"
-		)
-		(pin "30"
-		)
-		(pin "34"
-		)
-		(instances
-			(project ""
-				(path "/90bbffcf-f1b0-4966-a1ef-be58cceb8518"
-					(reference "J3")
-					(unit 1)
-				)
-			)
 		)
 	)
