File: LCD_Adapter/LCD_Adapter_HAT/STM2LCD.kicad_sch (KiCad schematic)
At the start: 24 parts, among them J2 FH12-30S-0.5SH_55_, J6 2-1734248-0, Q1 2N7002, Q2 2N7002

Commit message: UPDATE
Parts:
- removed R1: 0, Resistor_SMD:R_0603_1608Metric, symbol Device:R
- added C10, C11, C9: 0.47uF, Capacitor_SMD:C_0603_1608Metric, symbol Device:C
- added J3: RPi_GPIO, lib:RPI_Hat_B+, symbol RPi_Hat:RPi_GPIO
- added R21, R22: 1k, Resistor_SMD:R_0603_1608Metric, symbol Device:R
- added R23: 200k, Resistor_SMD:R_0603_1608Metric, symbol Device:R
- added R24, R25, R26, R27, R28: 0, Resistor_SMD:R_0603_1608Metric, symbol Device:R
- added TP1, TP15, TP16, TP5, TP6: TestPoint, TestPoint:TestPoint_Pad_D1.0mm, symbol Connector:TestPoint
- added U4: PCA9306DCURG4, PCA9306DCURG4:SOP50P310X90-8N, symbol PCA9306DCURG4:PCA9306DCURG4
- R6: value 10k -> 100k; LCSC# C25804 -> (none); now not fitted
Connections:
- net +1V8: now also C11.1, R21.2, R22.2, U4.2 (VREF1)
- net +2V8: now also C10.1
- net +3V3: now also C9.1, R23.2
- net DC_LED_PWM: now also R20.2, TP15.1
- net GND: now also C10.2, C11.2, C9.2, J3.14 (GND), J3.20 (GND), J3.25 (GND), J3.30 (GND), J3.34 (GND), J3.39 (GND), J3.6 (GND), J3.9 (GND), U4.1 (GND)
- net LCM_ID: now also R19.2
- net RESET: now also TP16.1
- net TP_INT: now also R11.2, TP1.1
- net TP_RES: now also TP5.1
- net TP_RES_STM_SIDE: now also R28.2
- net TP_SCL: now also R26.2
- net TP_SDA: now also R27.2
- net at R19.1: now also J3.16 (BCM23)
- net at R11.1: now also J3.18 (BCM24)
- net at R2.1: now also J3.37 (BCM26)
- net at Q1.1 (G), R3.2, R6.2: now also TP6.1
- net at J6.11, J6.31: now also R25.1
- net at J6.12, J6.32: now also R24.1
- net at R10.1: now also J3.32 (BCM12_PWM0)
- net at R20.1: now also J3.33 (BCM13_PWM1)
- new net: R21.1, R26.1, U4.3 (SCL1)
- new net: R25.2, U4.6 (SCL2)
- new net: R22.1, R27.1, U4.4 (SDA1)
- new net: J3.22 (BCM25), R28.1
- new net: R24.2, U4.5 (SDA2)
- new net: R23.1, U4.7 (VREF2), U4.8 (EN)
- no-connect marks 2 -> 0
Other:
- moved on the sheet: C13, C14, C15, C16, J2, J6, Q1, Q2, R10, R11, R19, R2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
