File: LCD_Adapter/LCD_Adapter_HAT/PWM.kicad_sch (KiCad schematic)
At the start: 28 parts, among them U1 TLV75801PDBV, U2 TLV75801PDBV, U3 TPS61042DRBR

Commit message: PCB_UPDATE
Parts:
- added R11: 6.8, Resistor_SMD:R_0603_1608Metric, symbol Device:R
- L1: LCSC # C703083 -> (none); LCSC# (none) -> C703083
- TP10, TP11, TP12, TP13, TP14, TP7, TP8, TP9: now left out of the parts list
Connections:
- net GND: no longer R16.1
